File: Synapse.sch (KiCad schematic (older format))
At the start: 32 parts, among them SW1 SW_SPST, SW2 SW_SPST, U4 STM32F411CEUx, U5 AMS1117-3.3, Y1 25MHz 9pF, Y2 32.768K 7pF

Commit message: PAUSED: Use `git resume` to continue working.
Parts:
- removed C26: 10n, Capacitor_SMD:C_0402_1005Metric, symbol Device:C_Small
- removed C31: 100n, Capacitor_SMD:C_0402_1005Metric, symbol Device:C_Small
- added C1, C12, C?: 100n, Capacitor_SMD:C_0402_1005Metric, symbol Device:C_Small
- added D1: LED, LED_SMD:LED_0603_1608Metric, symbol Device:LED
- added J1: Conn_01x04_Female, Connector_PinHeader_2.54mm:PinHeader_1x04_P2.54mm_Vertical, symbol Connector:Conn_01x04_Female
- added R1: 5.1K, Resistor_SMD:R_0603_1608Metric, symbol Device:R
- added U?: 24LC256, symbol Memory_EEPROM:24LC256
- C10: renamed from C20; value 4pF -> 4p
- C7: renamed from C17; value 8pF -> 8p
- C8: renamed from C18; value 8pF -> 8p
- C9: renamed from C19; value 4pF -> 4p
- R5: renamed from R8; footprint Resistor_SMD:R_0805_2012Metric -> Resistor_SMD:R_0402_1005Metric; LCSC C27834 -> C25905
- R6: renamed from R12; footprint Resistor_SMD:R_0805_2012Metric -> Resistor_SMD:R_0402_1005Metric; LCSC C27834 -> C25905
- SW1, SW2: footprint Button_Switch_SMD:SW_SPST_PTS645 -> Common:K2-1102SP-C4SC-04; LCSC C620316 -> C127509
- renumbered C24 to C11, C32 to C13, C23 to C14, C33 to C15, C28 to C16, C30 to C17, C21 to C2, C22 to C3, C25 to C4, C27 to C5, C29 to C6, L3 to L1, R15 to R2, R13 to R3, R14 to R4, U4 to U1, U5 to U2
Connections:
- net +BATT is gone; now on net +3V3: U1.1 (VBAT)
- net +3.3VA: now also C12.1
- net +3V3: now also C1.1, C?.2, J1.1 (Pin_1), R1.2, U?.8 (VCC)
- net GND: now also C1.2, C12.2, C?.1, D1.1 (K), J1.4 (Pin_4), U?.1 (A0), U?.2 (A1), U?.3 (A2), U?.4 (GND), U?.7 (WP)
- net I2C1_SCL: now also U?.6 (SCL)
- net I2C1_SDA: now also U?.5 (SDA)
- net SWDIO: now reaches U1.34 (PA13)
- net SWDIO: now also J1.2 (Pin_2)
- net SWCLK: now reaches U1.37 (PA14)
- net SWCLK: now also J1.3 (Pin_3)
- new net: D1.2 (A), R1.1
Other:
- note added: "Debug"
- note added: "EEPROM"
- note added: "Indicator light"
- note added: "RTC"
- note added: "TODO(ibash) double check\nthis inductor value"
- note removed: "TODO RTC circuit"
- note removed: "TODO SW Debug"
- note removed: "TODO(ibash) check if resistors can be smaller (instead of 805)"
- note removed: "TODO(ibash) check values here"
- moved on the sheet: C11, C15, L1, R4, R5, R6, SW2, USB1, USB2, USB3

Commit message: PAUSED: Use `git resume` to continue working.
Parts:
- added C?: 100pF ceramic, 100v, 10%, Capacitor_SMD:C_0805_2012Metric, symbol Device:C_Small
- added FB? (x2): 120Ω @ 100MHz, Inductor_SMD:L_0603_1608Metric, symbol Device:Ferrite_Bead_Small
- added Q?: Q_NMOS_GSD 1Amp, Package_TO_SOT_SMD:SOT-23, symbol Device:Q_NMOS_GSD
- added Q?: Q_PMOS_GSD, -3.6A 0.02R, Package_TO_SOT_SMD:SOT-23, symbol Device:Q_PMOS_GSD
- added R? (x2): 10k. 125mW. 5%., Resistor_SMD:R_0805_2012Metric, symbol Device:R_Small
- added R? (x2): 2.7K, Resistor_SMD:R_0805_2012Metric, symbol Device:R_Small
- added R? (x2): 200k, Resistor_SMD:R_0805_2012Metric, symbol Device:R_Small
- R?: renamed from R6; symbol Device:R -> Device:R_Small
- R?: renamed from R5; symbol Device:R -> Device:R_Small
- renumbered C12 to C?, C1 to C?, C7 to C?, C8 to C?, C9 to C?, C10 to C?, C2 to C?, C3 to C?, C4 to C?, C5 to C?, C6 to C?, C11 to C?, C14 to C?, C16 to C?, C17 to C?, C15 to C?, C13 to C?, D1 to D?, J1 to J?, L1 to L?, R1 to R?, R2 to R?, R4 to R?, R3 to R?, SW2 to SW?, SW1 to SW?, U1 to U?, U2 to U?, USB1 to USB?, USB2 to USB?, USB3 to USB?, Y1 to Y?, Y2 to Y?
Connections:
- net +5V: now also FB?.2, Q?.2 (S), R?.1, R?.1, R?.1
- net GND: now also USB?.A1 (GND), USB?.A12 (GND), USB?.B1 (GND), USB?.B12 (GND), USB?.S1 (SHIELD), R?.1, R?.1
- net I2C1_SCL: now also USB?.A6 (D+), USB?.B6 (D+), R?.2
- net I2C1_SDA: now also USB?.A7 (D-), USB?.B7 (D-), R?.2
- net SIDE_SWITCH: now reaches U?.21 (PB10)
- net SIDE_SWITCH: now also Q?.1 (G), R?.1
- net SIDE_POWER: now reaches USB?.A4 (VBUS), USB?.A9 (VBUS), USB?.B4 (VBUS), USB?.B9 (VBUS)
- net SIDE_POWER: now also USB?.A4 (VBUS), USB?.A9 (VBUS), USB?.B4 (VBUS), USB?.B9 (VBUS), FB?.1
- net at USB?.A5 (CC1): now also USB?.B5 (CC2), R?.2 (x2)
- net PB2 renamed BOOT1
- net VBUS: no longer names the net of USB?.A4 (VBUS), USB?.A9 (VBUS), USB?.B4 (VBUS), USB?.B9 (VBUS)
- net VBUS: now also FB?.1
- new net: Q?.1 (G), Q?.3 (D), R?.2
- new net: C?.1, FB?.2, Q?.3 (D)
- new net GNDREF: C?.2, Q?.2 (S), R?.2
- no-connect marks 0 -> 4
Other:
- note added: "I2C Pull ups"
- note added: "Side switch"
- note added: "pull down to ground > 126k\nindicates disabled"
- moved on the sheet: R?, U?

Commit message: PAUSED: Use `git resume` to continue working.
Parts:
- U3: renamed from U?; footprint (none) -> Package_SO:SOIC-8_3.9x4.9mm_P1.27mm
- gave numbers to parts that had none: 47

Commit message: PAUSED: Use `git resume` to continue working.
Parts:
- added D?: BLUE LED, LED_SMD:LED_0603_1608Metric, symbol Device:LED
- added R?: 1.5K, Resistor_SMD:R_0603_1608Metric, symbol Device:R
- D1: value LED -> RED LED
Connections:
- net +3V3: now also R?.2
- net PC13: now reaches U1.2 (PC13)
- net PC13: now also D?.1 (K)
- new net: D?.2 (A), R?.1
Changed lines of the file:
@@
 P 7650 2500
 F 0 "D1" H 7643 2245 50  0000 C CNN
-F 1 "LED" H 7643 2336 50  0000 C CNN
+F 1 "RED LED" H 7643 2336 50  0000 C CNN
 F 2 "LED_SMD:LED_0603_1608Metric" H 7650 2500 50  0001 C CNN
 F 3 "~" H 7650 2500 50  0001 C CNN
@@
 Text Notes 7250 5100 0    50   ~ 0
 I2C Pull ups
+$Comp
+L Device:R R?
+U 1 1 60F618A9
+P 7350 2950
+F 0 "R?" V 7143 2950 50  0000 C CNN
+F 1 "1.5K" V 7234 2950 50  0000 C CNN
+F 2 "Resistor_SMD:R_0603_1608Metric" V 7280 2950 50  0001 C CNN
+F 3 "~" H 7350 2950 50  0001 C CNN
+F 4 "C22843" V 7350 2950 50  0001 C CNN "LCSC"
+	1    7350 2950
+	0    1    1    0
+$EndComp
+$Comp
+L power:+3.3V #PWR?
+U 1 1 60F618AF
+P 7200 2950
+AR Path="/60F56179/60F618AF" Ref="#PWR?"  Part="1"
+AR Path="/60F618AF" Ref="#PWR?"  Part="1"
+F 0 "#PWR?" H 7200 2800 50  0001 C CNN
+F 1 "+3.3V" H 7200 3100 50  0000 C CNN
+F 2 "" H 7200 2950 50  0001 C CNN
+F 3 "" H 7200 2950 50  0001 C CNN
+	1    7200 2950
+	0    -1   -1   0
+$EndComp
+$Comp
+L Device:LED D?
+U 1 1 60F6189C
+P 7650 2950
+F 0 "D?" H 7643 2695 50  0000 C CNN
+F 1 "BLUE LED" H 7643 2786 50  0000 C CNN
+F 2 "LED_SMD:LED_0603_1608Metric" H 7650 2950 50  0001 C CNN
+F 3 "~" H 7650 2950 50  0001 C CNN
+F 4 "C72041" H 7650 2950 50  0001 C CNN "LCSC"
+	1    7650 2950
+	-1   0    0    1
+$EndComp
+Text GLabel 7800 2950 2    50   Input ~ 0
+PC13
+Text GLabel 1100 2000 0    50   Input ~ 0
+PC13
 $EndSCHEMATC

Commit message: PAUSED: Use `git resume` to continue working.
Parts:
- C1, C12, C13, C18, C19, C3, C4, C5, C6: LCSC (none) -> C1525; LCSC Part # C1525 -> (none)
- C10, C9: LCSC (none) -> C318615; LCSC Part # C318615 -> (none)
- C11: LCSC (none) -> C52923; LCSC Part # C52923 -> (none)
- C15, C16, C2: LCSC (none) -> C19666; LCSC Part # C19666 -> (none)
- C17: LCSC (none) -> C15195; LCSC Part # C15195 -> (none)
- C7, C8: LCSC (none) -> C26408; LCSC Part # C26408 -> (none)
- L1: LCSC (none) -> C26443; LCSC Part # C26443 -> (none)
- R2, R3: LCSC (none) -> C25744; LCSC Part # C25744 -> (none)
- R5: renamed from R4; LCSC (none) -> C25744; LCSC Part # C25744 -> (none)
- U1: LCSC (none) -> C60420
- U3: JCSC C6482 -> (none); LCSC (none) -> C6482
- Y1: LCSC (none) -> C390937; LCSC Part # C390937 -> (none)
- Y2: LCSC (none) -> C99009; LCSC Part # C99009 -> (none)
- gave numbers to parts that had none: 2
- renumbered R9 to R10, R10 to R11, R11 to R12, R12 to R13, R5 to R6, R6 to R7, R7 to R8, R8 to R9

Commit message: PAUSED: Use `git resume` to continue working.
Connections:
- no-connect marks 4 -> 30
Changed lines of the file:
@@
 Comment4 ""
 $EndDescr
-$Comp
-L MCU_ST_STM32F4:STM32F411CEUx U1
-U 1 1 60EF9182
-P 1800 2400
-F 0 "U1" H 1200 4100 50  0000 C CNN
-F 1 "STM32F411CEUx" H 1200 3950 50  0000 C CNN
-F 2 "Package_DFN_QFN:QFN-48-1EP_7x7mm_P0.5mm_EP5.6x5.6mm" H 1200 900 50  0001 R CNN
-F 3 "http://www.st.com/st-web-ui/static/active/en/resource/technical/document/datasheet/DM00115249.pdf" H 1800 2400 50  0001 C CNN
-F 4 "C60420" H 1800 2400 50  0001 C CNN "LCSC"
-	1    1800 2400
-	1    0    0    -1
-$EndComp
 Text GLabel 1100 3100 0    50   Input ~ 0
 I2C1_SDA
@@
 F 2 "Capacitor_SMD:C_0402_1005Metric" H 4462 2149 50  0001 C CNN
 F 3 "~" H 4462 2149 50  0001 C CNN
-F 4 "" H 4462 2149 50  0001 C CNN "LCSC Part #"
-F 5 "C318615" H 4462 2149 50  0001 C CNN "LCSC"
+F 4 "C318615" H 4462 2149 50  0001 C CNN "LCSC"
 	1    4462 2149
 	1    0    0    -1
@@
 F 2 "Resistor_SMD:R_0402_1005Metric" H 10050 2500 50  0001 C CNN
 F 3 "~" H 10050 2500 50  0001 C CNN
-F 4 "" H 10050 2500 50  0001 C CNN "LCSC Part #"
-F 5 "C25744" H 10050 2500 50  0001 C CNN "LCSC"
+F 4 "C25744" H 10050 2500 50  0001 C CNN "LCSC"
 	1    10050 2500
 	1    0    0    -1
@@
 F 2 "Capacitor_SMD:C_0603_1608Metric" H 6050 3600 50  0001 C CNN
 F 3 "~" H 6050 3600 50  0001 C CNN
-F 4 "" H 6050 3600 50  0001 C CNN "LCSC Part #"
-F 5 "C19666" H 6050 3600 50  0001 C CNN "LCSC"
+F 4 "C19666" H 6050 3600 50  0001 C CNN "LCSC"
 	1    6050 3600
 	1    0    0    -1
@@
 F 2 "Capacitor_SMD:C_0603_1608Metric" H 6850 3700 50  0001 C CNN
 F 3 "~" H 6850 3700 50  0001 C CNN
-F 4 "" H 6850 3700 50  0001 C CNN "LCSC Part #"
-F 5 "C19666" H 6850 3700 50  0001 C CNN "LCSC"
+F 4 "C19666" H 6850 3700 50  0001 C CNN "LCSC"
 	1    6850 3700
 	1    0    0    -1
@@
 F 2 "Capacitor_SMD:C_0402_1005Metric" H 7200 3700 50  0001 C CNN
 F 3 "~" H 7200 3700 50  0001 C CNN
-F 4 "" H 7200 3700 50  0001 C CNN "LCSC Part #"
-F 5 "C15195" H 7200 3700 50  0001 C CNN "LCSC"
+F 4 "C15195" H 7200 3700 50  0001 C CNN "LCSC"
 	1    7200 3700
 	1    0    0    -1
@@
 F 2 "Resistor_SMD:R_0402_1005Metric" H 9100 3250 50  0001 C CNN
 F 3 "~" H 9100 3250 50  0001 C CNN
-F 4 "" H 9100 3250 50  0001 C CNN "LCSC Part #"
-F 5 "C25744" H 9100 3250 50  0001 C CNN "LCSC"
+F 4 "C25744" H 9100 3250 50  0001 C CNN "LCSC"
 	1    9100 3250
 	1    0    0    -1
@@
 F 2 "Capacitor_SMD:C_0402_1005Metric" H 9450 3700 50  0001 C CNN
 F 3 "~" H 9450 3700 50  0001 C CNN
-F 4 "" H 9450 3700 50  0001 C CNN "LCSC Part #"
-F 5 "C1525" H 9450 3700 50  0001 C CNN "LCSC"
+F 4 "C1525" H 9450 3700 50  0001 C CNN "LCSC"
 	1    9450 3700
 	0    1    1    0
@@
 F 2 "Capacitor_SMD:C_0402_1005Metric" H 8900 2400 50  0001 C CNN
 F 3 "~" H 8900 2400 50  0001 C CNN
-F 4 "" H 8900 2400 50  0001 C CNN "LCSC Part #"
-F 5 "C1525" H 8900 2400 50  0001 C CNN "LCSC"
+F 4 "C1525" H 8900 2400 50  0001 C CNN "LCSC"
 	1    8900 2400
 	0    -1   -1   0
@@
 F 2 "Resistor_SMD:R_0402_1005Metric" H 8900 2650 50  0001 C CNN
 F 3 "~" H 8900 2650 50  0001 C CNN
-F 4 "" H 8900 2650 50  0001 C CNN "LCSC Part #"
-F 5 "C25744" H 8900 2650 50  0001 C CNN "LCSC"
+F 4 "C25744" H 8900 2650 50  0001 C CNN "LCSC"
 	1    8900 2650
 	0    1    1    0
@@
 F 2 "Crystal:Crystal_SMD_2012-2Pin_2.0x1.2mm" H 4712 1899 50  0001 C CNN
 F 3 "~" H 4712 1899 50  0001 C CNN
-F 4 "" H 4712 1899 50  0001 C CNN "LCSC Part #"
-F 5 "C99009" H 4712 1899 50  0001 C CNN "LCSC"
+F 4 "C99009" H 4712 1899 50  0001 C CNN "LCSC"
 	1    4712 1899
 	1    0    0    -1
@@
 F 2 "Capacitor_SMD:C_0402_1005Metric" H 4962 2149 50  0001 C CNN
 F 3 "~" H 4962 2149 50  0001 C CNN
-F 4 "" H 4962 2149 50  0001 C CNN "LCSC Part #"
-F 5 "C318615" H 4962 2149 50  0001 C CNN "LCSC"
+F 4 "C318615" H 4962 2149 50  0001 C CNN "LCSC"
 	1    4962 2149
 	1    0    0    -1
@@
 F 2 "Crystal:Crystal_SMD_2520-4Pin_2.5x2.0mm" H 3500 1800 50  0001 C CNN
 F 3 "~" H 3500 1800 50  0001 C CNN
-F 4 "" H 3500 1800 50  0001 C CNN "LCSC Part #"
-F 5 "C390937" H 3500 1800 50  0001 C CNN "LCSC"
+F 4 "C390937" H 3500 1800 50  0001 C CNN "LCSC"
 	1    3500 1800
 	1    0    0    -1
@@
 F 2 "Capacitor_SMD:C_0402_1005Metric" H 3750 2050 50  0001 C CNN
 F 3 "~" H 3750 2050 50  0001 C CNN
-F 4 "" H 3750 2050 50  0001 C CNN "LCSC Part #"
-F 5 "C26408" H 3750 2050 50  0001 C CNN "LCSC"
+F 4 "C26408" H 3750 2050 50  0001 C CNN "LCSC"
 	1    3750 2050
 	1    0    0    -1
@@
 F 2 "Capacitor_SMD:C_0402_1005Metric" H 3250 2050 50  0001 C CNN
 F 3 "~" H 3250 2050 50  0001 C CNN
-F 4 "" H 3250 2050 50  0001 C CNN "LCSC Part #"
-F 5 "C26408" H 3250 2050 50  0001 C CNN "LCSC"
+F 4 "C26408" H 3250 2050 50  0001 C CNN "LCSC"
 	1    3250 2050
 	1    0    0    -1
@@
 F 2 "Capacitor_SMD:C_0402_1005Metric" H 6050 1575 50  0001 C CNN
 F 3 "~" H 6050 1575 50  0001 C CNN
-F 4 "" H 6050 1575 50  0001 C CNN "LCSC Part #"
-F 5 "C1525" H 6050 1575 50  0001 C CNN "LCSC"
+F 4 "C1525" H 6050 1575 50  0001 C CNN "LCSC"
 	1    6050 1575
 	1    0    0    -1
@@
 F 2 "Capacitor_SMD:C_0402_1005Metric" H 6425 1575 50  0001 C CNN
 F 3 "~" H 6425 1575 50  0001 C CNN
-F 4 "" H 6425 1575 50  0001 C CNN "LCSC Part #"
-F 5 "C1525" H 6425 1575 50  0001 C CNN "LCSC"
+F 4 "C1525" H 6425 1575 50  0001 C CNN "LCSC"
 	1    6425 1575
 	1    0    0    -1
@@
 F 2 "Capacitor_SMD:C_0402_1005Metric" H 6800 1575 50  0001 C CNN
 F 3 "~" H 6800 1575 50  0001 C CNN
-F 4 "" H 6800 1575 50  0001 C CNN "LCSC Part #"
-F 5 "C1525" H 6800 1575 50  0001 C CNN "LCSC"
+F 4 "C1525" H 6800 1575 50  0001 C CNN "LCSC"
 	1    6800 1575
 	1    0    0    -1
@@
 F 2 "Capacitor_SMD:C_0402_1005Metric" H 7175 1575 50  0001 C CNN
 F 3 "~" H 7175 1575 50  0001 C CNN
-F 4 "" H 7175 1575 50  0001 C CNN "LCSC Part #"
-F 5 "C1525" H 7175 1575 50  0001 C CNN "LCSC"
+F 4 "C1525" H 7175 1575 50  0001 C CNN "LCSC"
 	1    7175 1575
 	1    0    0    -1
@@
 F 2 "Capacitor_SMD:C_0402_1005Metric" H 6100 2400 50  0001 C CNN
 F 3 "~" H 6100 2400 50  0001 C CNN
-F 4 "" H 6100 2400 50  0001 C CNN "LCSC Part #"
-F 5 "C52923" H 6100 2400 50  0001 C CNN "LCSC"
+F 4 "C52923" H 6100 2400 50  0001 C CNN "LCSC"
 	1    6100 2400
 	1    0    0    -1
@@
 F 2 "Inductor_SMD:L_0402_1005Metric" H 5900 2300 50  0001 C CNN
 F 3 "~" H 5900 2300 50  0001 C CNN
-F 4 "" H 5900 2300 50  0001 C CNN "LCSC Part #"
-F 5 "C26443" H 5900 2300 50  0001 C CNN "LCSC"
+F 4 "C26443" H 5900 2300 50  0001 C CNN "LCSC"
 	1    5900 2300
 	0    -1   -1   0
@@
 F 2 "Capacitor_SMD:C_0402_1005Metric" H 6400 2400 50  0001 C CNN
 F 3 "~" H 6400 2400 50  0001 C CNN
-F 4 "" H 6400 2400 50  0001 C CNN "LCSC Part #"
-F 5 "C1525" H 6400 2400 50  0001 C CNN "LCSC"
+F 4 "C1525" H 6400 2400 50  0001 C CNN "LCSC"
 	1    6400 2400
 	1    0    0    -1
@@
 F 2 "Capacitor_SMD:C_0603_1608Metric" H 5700 1575 50  0001 C CNN
 F 3 "~" H 5700 1575 50  0001 C CNN
-F 4 "" H 5700 1575 50  0001 C CNN "LCSC Part #"
-F 5 "C19666" H 5700 1575 50  0001 C CNN "LCSC"
+F 4 "C19666" H 5700 1575 50  0001 C CNN "LCSC"
 	1    5700 1575
 	1    0    0    -1
@@
 F 2 "Capacitor_SMD:C_0402_1005Metric" H 9050 1500 50  0001 C CNN
 F 3 "~" H 9050 1500 50  0001 C CNN
-F 4 "" H 9050 1500 50  0001 C CNN "LCSC Part #"
-F 5 "C1525" H 9050 1500 50  0001 C CNN "LCSC"
+F 4 "C1525" H 9050 1500 50  0001 C CNN "LCSC"
 	1    9050 1500
 	1    0    0    -1
@@
 F 2 "Capacitor_SMD:C_0402_1005Metric" H 8700 4650 50  0001 C CNN
 F 3 "~" H 8700 4650 50  0001 C CNN
-F 4 "" H 8700 4650 50  0001 C CNN "LCSC Part #"
-F 5 "C1525" H 8700 4650 50  0001 C CNN "LCSC"
+F 4 "C1525" H 8700 4650 50  0001 C CNN "LCSC"
 	1    8700 4650
 	-1   0    0    1
@@
 Text GLabel 1100 2000 0    50   Input ~ 0
 PC13
+NoConn ~ 2050 6300
+NoConn ~ 2050 6400
+NoConn ~ 1100 1500
+NoConn ~ 1100 2400
+NoConn ~ 1100 2500
+NoConn ~ 1100 2700
+NoConn ~ 1100 2800
+NoConn ~ 1100 2900
+NoConn ~ 2400 2300
+NoConn ~ 2400 2400
+NoConn ~ 2400 2500
+NoConn ~ 2400 2600
+NoConn ~ 2400 2700
+NoConn ~ 2400 2800
+NoConn ~ 2400 2900
+NoConn ~ 2400 3000
+NoConn ~ 2400 3100
+NoConn ~ 2400 3200
+NoConn ~ 2400 3300
+NoConn ~ 1100 3300
+NoConn ~ 1100 3200
+NoConn ~ 1100 3800
+NoConn ~ 1100 3700
+$Comp
+L MCU_ST_STM32F4:STM32F411CEUx U1
+U 1 1 60EF9182
+P 1800 2400
+F 0 "U1" H 1200 4100 50  0000 C CNN
+F 1 "STM32F411CEUx" H 1200 3950 50  0000 C CNN
+F 2 "Package_DFN_QFN:QFN-48-1EP_7x7mm_P0.5mm_EP5.6x5.6mm" H 1200 900 50  0001 R CNN
+F 3 "http://www.st.com/st-web-ui/static/active/en/resource/technical/document/datasheet/DM00115249.pdf" H 1800 2400 50  0001 C CNN
+F 4 "C60420" H 1800 2400 50  0001 C CNN "LCSC"
+	1    1800 2400
+	1    0    0    -1
+$EndComp
+NoConn ~ 1100 3600
+NoConn ~ 1100 3500
+NoConn ~ 2400 3800
 $EndSCHEMATC
