File: Synapse.sch (KiCad schematic (older format))
At the start: 50 parts, among them J1 Conn_01x04_Female, Q1 Q_PMOS_GSD, -3.6A 0.02R, Q2 Q_NMOS_GSD 1Amp, SW1 SW_SPST, SW2 SW_SPST, U1 STM32F411CEUx, U2 AMS1117-3.3, U3 24LC256, Y1 25MHz 9pF, Y2 32.768K 7pF

Commit message: PAUSED: Use `git resume` to continue working.
Parts:
- C14: value 100pF ceramic, 100v, 10% -> 100p; footprint Capacitor_SMD:C_0805_2012Metric -> Capacitor_SMD:C_0402_1005Metric; LCSC C159771 -> C1546
- D1: value RED LED -> Red LED
- D2: value BLUE LED -> Blue LED
- FB1, FB2: value 120Ω @ 100MHz -> 470 @ 100MHz; LCSC C85831 -> C97853
- FB?: renamed from L1; value 39n -> 470 @ 100MHz; footprint Inductor_SMD:L_0402_1005Metric -> Inductor_SMD:L_0603_1608Metric; symbol Device:L_Small -> Device:Ferrite_Bead_Small; LCSC C26443 -> C97853
- J1: LCSC (none) -> C85819
- R10, R9: footprint Resistor_SMD:R_0805_2012Metric -> Resistor_SMD:R_0402_1005Metric; LCSC C17539 -> C25764
- R12, R13: footprint Resistor_SMD:R_0805_2012Metric -> Resistor_SMD:R_0603_1608Metric; LCSC C17530 -> C13167
- R6, R7: value 10k. 125mW. 5%. -> 10k; footprint Resistor_SMD:R_0805_2012Metric -> Resistor_SMD:R_0402_1005Metric; LCSC C17414 -> C25744
Other:
- note removed: "TODO(ibash) double check\nthis inductor value"
- moved on the sheet: R6
Changed lines of the file:
@@
 $EndComp
 $Comp
-L Device:L_Small L?
+L Device:Ferrite_Bead_Small L?
 U 1 1 60FADF48
 P 5900 2300
 AR Path="/60F56179/60FADF48" Ref="L?"  Part="1"
-AR Path="/60FADF48" Ref="L1"  Part="1"
-F 0 "L1" V 5975 2300 50  0000 C CNN
-F 1 "39n" V 5825 2300 50  0000 C CNN
-F 2 "Inductor_SMD:L_0402_1005Metric" H 5900 2300 50  0001 C CNN
+AR Path="/60FADF48" Ref="FB?"  Part="1"
+F 0 "FB?" V 6050 2250 50  0000 C CNN
+F 1 "470 @ 100MHz" V 5825 2300 50  0001 C CNN
+F 2 "Inductor_SMD:L_0603_1608Metric" H 5900 2300 50  0001 C CNN
 F 3 "~" H 5900 2300 50  0001 C CNN
-F 4 "C26443" H 5900 2300 50  0001 C CNN "LCSC"
+F 4 "C97853" H 5900 2300 50  0001 C CNN "LCSC"
 	1    5900 2300
 	0    -1   -1   0
@@
 	1    0    0    -1
 $EndComp
-Text Notes 5900 2050 0    50   ~ 0
-TODO(ibash) double check\nthis inductor value
 Text Notes 8550 1050 0    50   ~ 0
 RTC
@@
 F 2 "Connector_PinHeader_2.54mm:PinHeader_1x04_P2.54mm_Vertical" H 9050 5800 50  0001 C CNN
 F 3 "~" H 9050 5800 50  0001 C CNN
+F 4 "C85819" H 9050 5800 50  0001 C CNN "LCSC"
 	1    9050 5800
 	1    0    0    -1
@@
 P 7650 2500
 F 0 "D1" H 7643 2245 50  0000 C CNN
-F 1 "RED LED" H 7643 2336 50  0000 C CNN
+F 1 "Red LED" H 7643 2336 50  0000 C CNN
 F 2 "LED_SMD:LED_0603_1608Metric" H 7650 2500 50  0001 C CNN
 F 3 "~" H 7650 2500 50  0001 C CNN
@@
 AR Path="/6105CA87" Ref="R7"  Part="1"
 F 0 "R7" H 4900 3950 50  0000 L CNN
-F 1 "10k. 125mW. 5%." H 4900 3850 50  0000 L CNN
-F 2 "Resistor_SMD:R_0805_2012Metric" V 4780 3950 50  0001 C CNN
+F 1 "10k" H 4900 3850 50  0000 L CNN
+F 2 "Resistor_SMD:R_0402_1005Metric" V 4780 3950 50  0001 C CNN
 F 3 "~" H 4850 3950 50  0001 C CNN
-F 4 "C17414" H 4850 3950 50  0001 C CNN "LCSC"
+F 4 "C25744" H 4850 3950 50  0001 C CNN "LCSC"
 	1    4850 3950
 	1    0    0    -1
@@
 L Device:R_Small R?
 U 1 1 6105CA8E
-P 4950 3450
+P 4850 3500
 AR Path="/6102A64B/6105CA8E" Ref="R?"  Part="1"
 AR Path="/6105CA8E" Ref="R6"  Part="1"
-F 0 "R6" H 5020 3496 50  0000 L CNN
-F 1 "10k. 125mW. 5%." H 5020 3405 50  0000 L CNN
-F 2 "Resistor_SMD:R_0805_2012Metric" V 4880 3450 50  0001 C CNN
-F 3 "~" H 4950 3450 50  0001 C CNN
-F 4 "C17414" H 4950 3450 50  0001 C CNN "LCSC"
-	1    4950 3450
+F 0 "R6" H 4920 3546 50  0000 L CNN
+F 1 "10k" H 4920 3455 50  0000 L CNN
+F 2 "Resistor_SMD:R_0402_1005Metric" V 4780 3500 50  0001 C CNN
+F 3 "~" H 4850 3500 50  0001 C CNN
+F 4 "C25744" H 4850 3500 50  0001 C CNN "LCSC"
+	1    4850 3500
 	1    0    0    -1
 $EndComp
@@
 AR Path="/6105CA95" Ref="FB1"  Part="1"
 F 0 "FB1" H 4000 3550 50  0000 L CNN
-F 1 "120Ω @ 100MHz" H 4000 3500 50  0001 L CNN
+F 1 "470 @ 100MHz" H 4000 3500 50  0001 L CNN
 F 2 "Inductor_SMD:L_0603_1608Metric" V 3830 3550 50  0001 C CNN
 F 3 "~" H 3900 3550 50  0001 C CNN
-F 4 "C85831" H 3900 3550 50  0001 C CNN "LCSC"
+F 4 "C97853" H 3900 3550 50  0001 C CNN "LCSC"
 	1    3900 3550
 	-1   0    0    1
@@
 L power:+5V #PWR?
 U 1 1 6105CA9B
-P 5200 3350
+P 5000 3350
 AR Path="/6102A64B/6105CA9B" Ref="#PWR?"  Part="1"
 AR Path="/6105CA9B" Ref="#PWR022"  Part="1"
-F 0 "#PWR022" H 5200 3200 50  0001 C CNN
-F 1 "+5V" H 5215 3523 50  0000 C CNN
-F 2 "" H 5200 3350 50  0001 C CNN
-F 3 "" H 5200 3350 50  0001 C CNN
-	1    5200 3350
+F 0 "#PWR022" H 5000 3200 50  0001 C CNN
+F 1 "+5V" H 5015 3523 50  0000 C CNN
+F 2 "" H 5000 3350 50  0001 C CNN
+F 3 "" H 5000 3350 50  0001 C CNN
+	1    5000 3350
 	1    0    0    -1
 $EndComp
@@
 Wire Wire Line
 	4550 3350 4350 3350
-Connection ~ 4950 3350
-Wire Wire Line
-	4950 3350 5200 3350
-Wire Wire Line
-	4750 3350 4950 3350
 Wire Wire Line
 	3900 3650 3900 3700
-Wire Wire Line
-	4550 3650 4950 3650
-Wire Wire Line
-	4950 3550 4950 3650
 Connection ~ 4550 3650
 $Comp
@@
 AR Path="/6105CAB8" Ref="C14"  Part="1"
 F 0 "C14" H 4265 3396 50  0000 L CNN
-F 1 "100pF ceramic, 100v, 10%" H 4265 3305 50  0000 L CNN
-F 2 "Capacitor_SMD:C_0805_2012Metric" H 4188 3200 50  0001 C CNN
+F 1 "100p" H 4265 3305 50  0000 L CNN
+F 2 "Capacitor_SMD:C_0402_1005Metric" H 4188 3200 50  0001 C CNN
 F 3 "~" H 4150 3350 50  0001 C CNN
-F 4 "C159771" H 4150 3350 50  0001 C CNN "LCSC"
+F 4 "C1546" H 4150 3350 50  0001 C CNN "LCSC"
 	1    4150 3350
 	-1   0    0    1
@@
 Text Notes 3850 3000 0    50   ~ 0
 Side switch
-Text GLabel 4850 3850 2    50   Input ~ 0
-SIDE_SWITCH
 Text GLabel 3900 3700 0    50   Input ~ 0
 SIDE_POWER
@@
 AR Path="/6106F684" Ref="FB2"  Part="1"
 F 0 "FB2" H 1950 5100 50  0000 L CNN
-F 1 "120Ω @ 100MHz" H 1400 4950 50  0001 L CNN
+F 1 "470 @ 100MHz" H 1400 4950 50  0001 L CNN
 F 2 "Inductor_SMD:L_0603_1608Metric" V 2130 5100 50  0001 C CNN
 F 3 "~" H 2200 5100 50  0001 C CNN
-F 4 "C85831" H 2200 5100 50  0001 C CNN "LCSC"
+F 4 "C97853" H 2200 5100 50  0001 C CNN "LCSC"
 	1    2200 5100
 	-1   0    0    1
@@
 F 0 "R13" H 7870 5596 50  0000 L CNN
 F 1 "2.7K" H 7870 5505 50  0000 L CNN
-F 2 "Resistor_SMD:R_0805_2012Metric" V 7730 5550 50  0001 C CNN
+F 2 "Resistor_SMD:R_0603_1608Metric" V 7730 5550 50  0001 C CNN
 F 3 "~" H 7800 5550 50  0001 C CNN
-F 4 "C17530" H 7800 5550 50  0001 C CNN "LCSC"
+F 4 "C13167" H 7800 5550 50  0001 C CNN "LCSC"
 	1    7800 5550
 	1    0    0    -1
@@
 F 0 "R12" H 7420 5596 50  0000 L CNN
 F 1 "2.7K" H 7420 5505 50  0000 L CNN
-F 2 "Resistor_SMD:R_0805_2012Metric" V 7280 5550 50  0001 C CNN
+F 2 "Resistor_SMD:R_0603_1608Metric" V 7280 5550 50  0001 C CNN
 F 3 "~" H 7350 5550 50  0001 C CNN
-F 4 "C17530" H 7350 5550 50  0001 C CNN "LCSC"
+F 4 "C13167" H 7350 5550 50  0001 C CNN "LCSC"
 	1    7350 5550
 	1    0    0    -1
@@
 F 0 "R9" V 3850 5400 50  0000 L CNN
 F 1 "200k" V 4050 5350 50  0000 L CNN
-F 2 "Resistor_SMD:R_0805_2012Metric" V 3880 5450 50  0001 C CNN
+F 2 "Resistor_SMD:R_0402_1005Metric" V 3880 5450 50  0001 C CNN
 F 3 "~" H 3950 5450 50  0001 C CNN
-F 4 "C17539" H 3950 5450 50  0001 C CNN "LCSC"
+F 4 "C25764" H 3950 5450 50  0001 C CNN "LCSC"
 	1    3950 5450
 	0    1    1    0
@@
 F 0 "R10" V 5500 5400 50  0000 L CNN
 F 1 "200k" V 5700 5350 50  0000 L CNN
-F 2 "Resistor_SMD:R_0805_2012Metric" V 5530 5450 50  0001 C CNN
+F 2 "Resistor_SMD:R_0402_1005Metric" V 5530 5450 50  0001 C CNN
 F 3 "~" H 5600 5450 50  0001 C CNN
-F 4 "C17539" H 5600 5450 50  0001 C CNN "LCSC"
+F 4 "C25764" H 5600 5450 50  0001 C CNN "LCSC"
 	1    5600 5450
 	0    1    1    0
@@
 P 7650 2950
 F 0 "D2" H 7643 2695 50  0000 C CNN
-F 1 "BLUE LED" H 7643 2786 50  0000 C CNN
+F 1 "Blue LED" H 7643 2786 50  0000 C CNN
 F 2 "LED_SMD:LED_0603_1608Metric" H 7650 2950 50  0001 C CNN
 F 3 "~" H 7650 2950 50  0001 C CNN
@@
 NoConn ~ 1100 3500
 NoConn ~ 2400 3800
+Text GLabel 4850 3850 2    50   Input ~ 0
+SIDE_SWITCH
+Wire Wire Line
+	4850 3350 4850 3400
+Connection ~ 4850 3350
+Wire Wire Line
+	4750 3350 4850 3350
+Wire Wire Line
+	4850 3650 4850 3600
+Wire Wire Line
+	4550 3650 4850 3650
+Wire Wire Line
+	4850 3350 5000 3350
 $EndSCHEMATC
