File: Synapse.sch (KiCad schematic (older format))
At the start: 50 parts, among them J1 Conn_01x04_Female, Q1 Q_PMOS_GSD, -3.6A 0.02R, Q2 Q_NMOS_GSD 1Amp, SW1 SW_SPST, SW2 SW_SPST, U1 STM32F411CEUx, U2 AMS1117-3.3, U3 24LC256, Y1 25MHz 9pF, Y2 32.768K 7pF

Commit message: PAUSED: Use `git resume` to continue working.
Parts:
- gave numbers to parts that had none: 1
- renumbered FB1 to FB2, FB2 to FB3
Changed lines of the file:
@@
 $EndComp
 $Comp
-L Device:Ferrite_Bead_Small L?
+L Device:Ferrite_Bead_Small FB?
 U 1 1 60FADF48
 P 5900 2300
-AR Path="/60F56179/60FADF48" Ref="L?"  Part="1"
-AR Path="/60FADF48" Ref="FB?"  Part="1"
-F 0 "FB?" V 6050 2250 50  0000 C CNN
+AR Path="/60F56179/60FADF48" Ref="FB?"  Part="1"
+AR Path="/60FADF48" Ref="FB1"  Part="1"
+F 0 "FB1" V 6050 2250 50  0000 C CNN
 F 1 "470 @ 100MHz" V 5825 2300 50  0001 C CNN
 F 2 "Inductor_SMD:L_0603_1608Metric" H 5900 2300 50  0001 C CNN
@@
 P 3900 3550
 AR Path="/6102A64B/6105CA95" Ref="FB?"  Part="1"
-AR Path="/6105CA95" Ref="FB1"  Part="1"
-F 0 "FB1" H 4000 3550 50  0000 L CNN
+AR Path="/6105CA95" Ref="FB2"  Part="1"
+F 0 "FB2" H 4000 3550 50  0000 L CNN
 F 1 "470 @ 100MHz" H 4000 3500 50  0001 L CNN
 F 2 "Inductor_SMD:L_0603_1608Metric" V 3830 3550 50  0001 C CNN
@@
 P 2200 5100
 AR Path="/6102A64B/6106F684" Ref="FB?"  Part="1"
-AR Path="/6106F684" Ref="FB2"  Part="1"
-F 0 "FB2" H 1950 5100 50  0000 L CNN
+AR Path="/6106F684" Ref="FB3"  Part="1"
+F 0 "FB3" H 1950 5100 50  0000 L CNN
 F 1 "470 @ 100MHz" H 1400 4950 50  0001 L CNN
 F 2 "Inductor_SMD:L_0603_1608Metric" V 2130 5100 50  0001 C CNN

Commit message: PAUSED: Use `git resume` to continue working.
Parts:
- added R1: 330, Resistor_SMD:R_0402_1005Metric, symbol Device:R_Small
- C10, C9: value 4p -> 15p; LCSC C318615 -> C1548
- C7, C8: value 8p -> 15p; LCSC C26408 -> C1548
- Y1: value 25MHz 9pF -> 25MHz 12pF; footprint Crystal:Crystal_SMD_2520-4Pin_2.5x2.0mm -> Crystal:Crystal_SMD_3225-4Pin_3.2x2.5mm; symbol Device:Crystal_Small -> Device:Crystal_GND24_Small; LCSC C390937 -> C9006
- Y2: value 32.768K 7pF -> 32.768K 12.5p; footprint Crystal:Crystal_SMD_2012-2Pin_2.0x1.2mm -> Crystal:Crystal_SMD_3215-2Pin_3.2x1.5mm; LCSC C99009 -> C32346
- renumbered R9 to R10, R10 to R11, R11 to R12, R12 to R13, R13 to R14, R1 to R2, R2 to R3, R3 to R4, R4 to R5, R5 to R6, R6 to R7, R7 to R8, R8 to R9
Connections:
- net HSE_IN: now also R1.1; no longer C8.1, Y1.2
- new net: C8.1, R1.2, Y1.3
Other:
- note added: "TODO(ibash) double check resistor values for leds"

Commit message: PAUSED: Use `git resume` to continue working.
Parts:
- removed C6: 100n, Capacitor_SMD:C_0402_1005Metric, symbol Device:C_Small
- removed R1: 330, Resistor_SMD:R_0402_1005Metric, symbol Device:R_Small
- added C14: 1u, Capacitor_SMD:C_0402_1005Metric, symbol Device:C_Small
- C15: value 4u7 -> 1u; footprint Capacitor_SMD:C_0603_1608Metric -> Capacitor_SMD:C_0402_1005Metric; LCSC C19666 -> C52923
- C2: value 4u7 -> 10u; LCSC C19666 -> C15525
- C6: renamed from C7; value 15p -> 6.8p; LCSC C1548 -> C1576
- C7: renamed from C8; value 15p -> 6.8p; LCSC C1548 -> C1576
- C8: renamed from C9; value 15p -> 2.7p; LCSC C1548 -> C1561
- C9: renamed from C10; value 15p -> 2.7p; LCSC C1548 -> C1561
- U2: value AMS1117-3.3 -> SOT-23-3 LDO; footprint Package_TO_SOT_SMD:SOT-223-3_TabPin2 -> Package_TO_SOT_SMD:SOT-23; LCSC C347222 -> C5446
- Y1: value 25MHz 12pF -> 25MHz 9pF; footprint Crystal:Crystal_SMD_3225-4Pin_3.2x2.5mm -> Crystal:Crystal_SMD_2520-4Pin_2.5x2.0mm; LCSC C9006 -> C390937
- Y2: value 32.768K 12.5p -> 32.768K 7p; footprint Crystal:Crystal_SMD_3215-2Pin_3.2x1.5mm -> Crystal:Crystal_SMD_2012-2Pin_2.0x1.2mm; LCSC C32346 -> C99009
- renumbered C11 to C10, C12 to C11, C13 to C12, C14 to C13, C18 to C16, C16 to C17, C17 to C18, R2 to R1, R11 to R10, R12 to R11, R13 to R12, R14 to R13, R3 to R2, R4 to R3, R5 to R4, R6 to R5, R7 to R6, R8 to R7, R9 to R8, R10 to R9
Connections:
- net GNDREF is gone; now on net GND: C13.2, Q2.2 (S), R7.2
- net +3V3: now also C15.1; no longer C17.1, C18.1
- net +5V: now also C14.1; no longer C15.1
- net GND: now also Y1.2, Y1.4, C14.2; no longer C17.2, C18.2
- net HSE_IN: now also C7.1, Y1.3
Other:
- note added: "Make this 10uf"
- moved on the sheet: C17, C18

Commit message: PAUSED: Use `git resume` to continue working.
Parts:
- removed J1: Conn_01x04_Female, Connector_PinHeader_2.54mm:PinHeader_1x04_P2.54mm_Vertical, symbol Connector:Conn_01x04_Female
- added TP? (x4): TestPoint, symbol Connector:TestPoint
- renumbered C11 to C?, C1 to C?, C6 to C?, C7 to C?, C8 to C?, C9 to C?, C2 to C?, C3 to C?, C4 to C?, C5 to C?, C19 to C?, C10 to C?, C17 to C?, C18 to C?, C16 to C?, C13 to C?, C12 to C?, C14 to C?, C15 to C?, D2 to D?, D1 to D?, FB1 to FB?, FB2 to FB?, FB3 to FB?, Q2 to Q?, Q1 to Q?, R4 to R?, R1 to R?, R2 to R?, R5 to R?, R7 to R?, R6 to R?, R3 to R?, R13 to R?, R12 to R?, R9 to R?, R11 to R?, R8 to R?, R10 to R?, SW2 to SW?, SW1 to SW?, U1 to U?, U3 to U?, U2 to U?, USB1 to USB?, USB2 to USB?, USB3 to USB?, Y1 to Y?, Y2 to Y?
Connections:
- net +3V3: now also TP?.1
- net GND: now also TP?.1
- net SWCLK: now also TP?.1
- net SWDIO: now also TP?.1

Commit message: PAUSED: Use `git resume` to continue working.
Parts:
- removed C?: 4u7, Capacitor_SMD:C_0603_1608Metric, symbol Device:C_Small
- removed C?: 10n, Capacitor_SMD:C_0402_1005Metric, symbol Device:C_Small
- removed TP? (x4): TestPoint, symbol Connector:TestPoint
- added J1: Conn_01x04_Female, Connector_PinHeader_2.54mm:PinHeader_1x04_P2.54mm_Vertical, symbol Connector:Conn_01x04_Female
- SW1, SW2: renamed from SW?; footprint Common:K2-1102SP-C4SC-04 -> Button_Switch_SMD:SW_SPST_B3U-1000P; LCSC C127509 -> C231329
- gave numbers to parts that had none: 45
Connections:
- net +3V3: now also J1.1 (Pin_1)
- net GND: now also J1.4 (Pin_4)
- net SWCLK: now also J1.3 (Pin_3)
- net SWDIO: now also J1.2 (Pin_2)
Other:
- note added: "Analog power filtering\n"
- note added: "Power conversion"
- note added: "Power filtering"
- note removed: "Make this 10uf"
- note removed: "Power"
- note removed: "Power Conversion"
- moved on the sheet: C10, C11, C13, C14, C15, C2, C3, C4, C5, FB1, FB2, Q1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

Commit message: PAUSED: Use `git resume` to continue working.
Other:
- moved on the sheet: C13, FB2
Changed lines of the file:
@@
 	1    0    0    -1
 $EndComp
-Wire Wire Line
-	4150 3100 3950 3100
-Wire Wire Line
-	3500 3400 3500 3450
 Connection ~ 4150 3400
-$Comp
-L power:GND #PWR?
-U 1 1 6105CABE
-P 3750 3000
-AR Path="/6102A64B/6105CABE" Ref="#PWR?"  Part="1"
-AR Path="/6105CABE" Ref="#PWR021"  Part="1"
-F 0 "#PWR021" H 3750 2750 50  0001 C CNN
-F 1 "GND" H 3755 2827 50  0001 C CNN
-F 2 "" H 3750 3000 50  0001 C CNN
-F 3 "" H 3750 3000 50  0001 C CNN
-	1    3750 3000
-	-1   0    0    1
-$EndComp
-Wire Wire Line
-	3750 3200 3950 3200
-Wire Wire Line
-	3950 3200 3950 3100
-Connection ~ 3950 3100
 Text Notes 3450 2750 0    50   ~ 0
 Side switch
-Text GLabel 3500 3450 0    50   Input ~ 0
-SIDE_POWER
 Wire Wire Line
 	2050 5200 2200 5200
@@
 	1    0    0    -1
 $EndComp
-Wire Wire Line
-	3500 3200 3750 3200
-Connection ~ 3750 3200
 Text GLabel 3850 5200 2    50   Input ~ 0
 SIDE_POWER
@@
 $Comp
 L Device:Ferrite_Bead_Small FB?
-U 1 1 6105CA95
-P 3500 3300
-AR Path="/6102A64B/6105CA95" Ref="FB?"  Part="1"
-AR Path="/6105CA95" Ref="FB2"  Part="1"
-F 0 "FB2" H 3600 3300 50  0000 L CNN
-F 1 "470 @ 100MHz" H 3600 3250 50  0001 L CNN
-F 2 "Inductor_SMD:L_0603_1608Metric" V 3430 3300 50  0001 C CNN
-F 3 "~" H 3500 3300 50  0001 C CNN
-F 4 "C97853" H 3500 3300 50  0001 C CNN "LCSC"
-	1    3500 3300
-	-1   0    0    1
-$EndComp
-$Comp
-L Device:C_Small C?
-U 1 1 6105CAB8
-P 3750 3100
-AR Path="/6102A64B/6105CAB8" Ref="C?"  Part="1"
-AR Path="/6105CAB8" Ref="C13"  Part="1"
-F 0 "C13" H 3865 3146 50  0000 L CNN
-F 1 "100p" H 3865 3055 50  0000 L CNN
-F 2 "Capacitor_SMD:C_0402_1005Metric" H 3788 2950 50  0001 C CNN
-F 3 "~" H 3750 3100 50  0001 C CNN
-F 4 "C1546" H 3750 3100 50  0001 C CNN "LCSC"
-	1    3750 3100
-	-1   0    0    1
-$EndComp
-$Comp
-L Device:Ferrite_Bead_Small FB?
 U 1 1 6106F684
 P 2200 5100
@@
 	1    0    0    -1
 $EndComp
+$Comp
+L Device:Ferrite_Bead_Small FB?
+U 1 1 6105CA95
+P 3500 3100
+AR Path="/6102A64B/6105CA95" Ref="FB?"  Part="1"
+AR Path="/6105CA95" Ref="FB2"  Part="1"
+F 0 "FB2" H 3600 3100 50  0000 L CNN
+F 1 "470 @ 100MHz" H 3600 3050 50  0001 L CNN
+F 2 "Inductor_SMD:L_0603_1608Metric" V 3430 3100 50  0001 C CNN
+F 3 "~" H 3500 3100 50  0001 C CNN
+F 4 "C97853" H 3500 3100 50  0001 C CNN "LCSC"
+	1    3500 3100
+	0    -1   -1   0
+$EndComp
+Text GLabel 3400 3100 0    50   Input ~ 0
+SIDE_POWER
+$Comp
+L power:GND #PWR?
+U 1 1 6105CABE
+P 3700 3300
+AR Path="/6102A64B/6105CABE" Ref="#PWR?"  Part="1"
+AR Path="/6105CABE" Ref="#PWR021"  Part="1"
+F 0 "#PWR021" H 3700 3050 50  0001 C CNN
+F 1 "GND" H 3705 3127 50  0001 C CNN
+F 2 "" H 3700 3300 50  0001 C CNN
+F 3 "" H 3700 3300 50  0001 C CNN
+	1    3700 3300
+	1    0    0    -1
+$EndComp
+$Comp
+L Device:C_Small C?
+U 1 1 6105CAB8
+P 3700 3200
+AR Path="/6102A64B/6105CAB8" Ref="C?"  Part="1"
+AR Path="/6105CAB8" Ref="C13"  Part="1"
+F 0 "C13" H 3800 3200 50  0000 L CNN
+F 1 "100p" H 3800 3100 50  0000 L CNN
+F 2 "Capacitor_SMD:C_0402_1005Metric" H 3738 3050 50  0001 C CNN
+F 3 "~" H 3700 3200 50  0001 C CNN
+F 4 "C1546" H 3700 3200 50  0001 C CNN "LCSC"
+	1    3700 3200
+	1    0    0    -1
+$EndComp
+Wire Wire Line
+	3600 3100 3700 3100
+Connection ~ 3700 3100
+Wire Wire Line
+	3700 3100 3950 3100
 $EndSCHEMATC

Commit message: PAUSED: Use `git resume` to continue working.
Parts:
- J1: value Conn_01x04_Female -> SWD; footprint Connector_PinHeader_2.54mm:PinHeader_1x04_P2.54mm_Vertical -> Common:TestPoint_Pads_4x2.54_D1.5mm
Connections:
- net +3V3: now also J1.4 (Pin_4); no longer J1.1 (Pin_1)
- net GND: now also J1.1 (Pin_1); no longer J1.4 (Pin_4)
- net SWCLK: now also J1.2 (Pin_2); no longer J1.3 (Pin_3)
- net SWDIO: now also J1.3 (Pin_3); no longer J1.2 (Pin_2)
Changed lines of the file:
@@
 L power:GND #PWR044
 U 1 1 60F704A2
-P 8850 6250
-F 0 "#PWR044" H 8850 6000 50  0001 C CNN
-F 1 "GND" H 8850 6100 50  0000 C CNN
-F 2 "" H 8850 6250 50  0001 C CNN
-F 3 "" H 8850 6250 50  0001 C CNN
-	1    8850 6250
+P 8850 5650
+F 0 "#PWR044" H 8850 5400 50  0001 C CNN
+F 1 "GND" H 8850 5500 50  0000 C CNN
+F 2 "" H 8850 5650 50  0001 C CNN
+F 3 "" H 8850 5650 50  0001 C CNN
+	1    8850 5650
 	0    1    1    0
 $EndComp
+Text GLabel 8850 6050 0    50   Input ~ 0
+SWDIO
 Text GLabel 8850 5850 0    50   Input ~ 0
-SWDIO
-Text GLabel 8850 6050 0    50   Input ~ 0
 SWCLK
 Text GLabel 2400 3600 2    50   Input ~ 0
@@
 	1    8700 4950
 	1    0    0    -1
-$EndComp
-$Comp
-L power:+3.3V #PWR?
-U 1 1 60F6F805
-P 8850 5650
-AR Path="/60F56179/60F6F805" Ref="#PWR?"  Part="1"
-AR Path="/60F6F805" Ref="#PWR043"  Part="1"
-F 0 "#PWR043" H 8850 5500 50  0001 C CNN
-F 1 "+3.3V" H 8850 5800 50  0000 C CNN
-F 2 "" H 8850 5650 50  0001 C CNN
-F 3 "" H 8850 5650 50  0001 C CNN
-	1    8850 5650
-	0    -1   1    0
 $EndComp
 $Comp
@@
 P 9250 5900
 F 0 "J1" H 9278 5876 50  0000 L CNN
-F 1 "Conn_01x04_Female" H 9278 5785 50  0000 L CNN
-F 2 "Connector_PinHeader_2.54mm:PinHeader_1x04_P2.54mm_Vertical" H 9250 5900 50  0001 C CNN
+F 1 "SWD" H 9278 5785 50  0000 L CNN
+F 2 "Common:TestPoint_Pads_4x2.54_D1.5mm" H 9250 5900 50  0001 C CNN
 F 3 "~" H 9250 5900 50  0001 C CNN
 	1    9250 5900
@@
 Wire Wire Line
 	3700 3100 3950 3100
+$Comp
+L power:+3.3V #PWR?
+U 1 1 60F6F805
+P 8850 6250
+AR Path="/60F56179/60F6F805" Ref="#PWR?"  Part="1"
+AR Path="/60F6F805" Ref="#PWR043"  Part="1"
+F 0 "#PWR043" H 8850 6100 50  0001 C CNN
+F 1 "+3.3V" H 8850 6400 50  0000 C CNN
+F 2 "" H 8850 6250 50  0001 C CNN
+F 3 "" H 8850 6250 50  0001 C CNN
+	1    8850 6250
+	0    -1   1    0
+$EndComp
 $EndSCHEMATC

Commit message: PAUSED: Use `git resume` to continue working.
Parts:
- removed D2: Blue LED, LED_SMD:LED_0603_1608Metric, symbol Device:LED
- removed R4: 1.5K, Resistor_SMD:R_0603_1608Metric, symbol Device:R
- D1: symbol Device:LED -> Device:LED_Small
- FB1, FB2, FB3: footprint Inductor_SMD:L_0603_1608Metric -> Inductor_SMD:L_0402_1005Metric; LCSC C97853 -> C333978
- Q1: footprint Package_TO_SOT_SMD:SOT-23 -> Package_TO_SOT_SMD:SOT-883; LCSC C15127 -> C146297
- Q2: footprint Package_TO_SOT_SMD:SOT-23 -> Package_TO_SOT_SMD:SOT-723; LCSC C20917 -> C110712
- R1: value 5.1K -> 1K; footprint Resistor_SMD:R_0603_1608Metric -> Resistor_SMD:R_0402_1005Metric; symbol Device:R -> Device:R_Small; LCSC C23186 -> C11702
- R12, R13: footprint Resistor_SMD:R_0603_1608Metric -> Resistor_SMD:R_0402_1005Metric; LCSC C13167 -> C25885
- U2: footprint Package_TO_SOT_SMD:SOT-23 -> Package_TO_SOT_SMD:SOT-553; LCSC C5446 -> C146430
Connections:
- net +3V3: now also D1.2 (A); no longer R1.2
- net GND: now also R1.1; no longer D1.1 (K)
- net SIDE_SWITCH: now also U1.25 (PB12); no longer U1.21 (PB10)
- net SWCLK: now also J1.3 (Pin_3); no longer J1.2 (Pin_2)
- net SWDIO: now also J1.2 (Pin_2); no longer J1.3 (Pin_3)
- net PC13: no longer names the net of U1.2 (PC13)
- new net: D1.1 (K), R1.2
- no-connect marks 30 -> 31
Other:
- moved on the sheet: D1, R1
Changed lines of the file:
@@
 	0    1    1    0
 $EndComp
-Text GLabel 8850 6050 0    50   Input ~ 0
-SWDIO
-Text GLabel 8850 5850 0    50   Input ~ 0
-SWCLK
 Text GLabel 2400 3600 2    50   Input ~ 0
 SWDIO
@@
 Debug
 $Comp
-L power:GND #PWR?
-U 1 1 60F7E24C
-P 7800 2500
-AR Path="/60F56179/60F7E24C" Ref="#PWR?"  Part="1"
-AR Path="/60F7E24C" Ref="#PWR015"  Part="1"
-F 0 "#PWR015" H 7800 2250 50  0001 C CNN
-F 1 "GND" H 7800 2350 50  0000 C CNN
-F 2 "" H 7800 2500 50  0001 C CNN
-F 3 "" H 7800 2500 50  0001 C CNN
-	1    7800 2500
-	0    -1   -1   0
-$EndComp
-$Comp
 L power:+3.3V #PWR?
 U 1 1 60F83F1E
-P 7200 2500
+P 7250 2350
 AR Path="/60F56179/60F83F1E" Ref="#PWR?"  Part="1"
 AR Path="/60F83F1E" Ref="#PWR014"  Part="1"
-F 0 "#PWR014" H 7200 2350 50  0001 C CNN
-F 1 "+3.3V" H 7200 2650 50  0000 C CNN
-F 2 "" H 7200 2500 50  0001 C CNN
-F 3 "" H 7200 2500 50  0001 C CNN
-	1    7200 2500
-	0    -1   -1   0
+F 0 "#PWR014" H 7250 2200 50  0001 C CNN
+F 1 "+3.3V" H 7250 2500 50  0000 C CNN
+F 2 "" H 7250 2350 50  0001 C CNN
+F 3 "" H 7250 2350 50  0001 C CNN
+	1    7250 2350
+	1    0    0    -1
 $EndComp
 Text Notes 7000 2150 0    50   ~ 0
@@
 Text Notes 5950 5500 0    50   ~ 0
 pull down to ground > 126k\nindicates disabled
-Text GLabel 1100 3400 0    50   Input ~ 0
+Text GLabel 1100 3500 0    50   Input ~ 0
 SIDE_SWITCH
 Connection ~ 3850 5450
@@
 NoConn ~ 1100 3700
 NoConn ~ 1100 3600
-NoConn ~ 1100 3500
+NoConn ~ 1100 3400
 NoConn ~ 2400 3800
 Text GLabel 4450 3600 2    50   Input ~ 0
@@
 F 0 "U2" H 5900 3292 50  0000 C CNN
 F 1 "SOT-23-3 LDO" H 5900 3201 50  0000 C CNN
-F 2 "Package_TO_SOT_SMD:SOT-23" H 5900 3250 50  0001 C CNN
+F 2 "Package_TO_SOT_SMD:SOT-553" H 5900 3250 50  0001 C CNN
 F 3 "" H 6000 2800 50  0001 C CNN
-F 4 "C5446" H 5900 3050 50  0001 C CNN "LCSC"
+F 4 "C146430" H 5900 3050 50  0001 C CNN "LCSC"
 	1    5900 3050
 	1    0    0    -1
@@
 P 2150 5500
 F 0 "R11" V 2250 5450 50  0000 C CNN
-F 1 "5.1K" V 2250 5600 50  0000 C CNN
+F 1 "5.1K" V 2250 5650 50  0000 C CNN
 F 2 "Resistor_SMD:R_0402_1005Metric" V 2080 5500 50  0001 C CNN
 F 3 "~" H 2150 5500 50  0001 C CNN
@@
 F 0 "FB1" V 7450 1300 50  0000 C CNN
 F 1 "470 @ 100MHz" V 7225 1350 50  0001 C CNN
-F 2 "Inductor_SMD:L_0603_1608Metric" H 7300 1350 50  0001 C CNN
+F 2 "Inductor_SMD:L_0402_1005Metric" H 7300 1350 50  0001 C CNN
 F 3 "~" H 7300 1350 50  0001 C CNN
-F 4 "C97853" H 7300 1350 50  0001 C CNN "LCSC"
+F 4 "C333978" H 7300 1350 50  0001 C CNN "LCSC"
 	1    7300 1350
 	0    -1   -1   0
@@
 $EndComp
 $Comp
-L Device:LED D1
+L Device:LED_Small D1
 U 1 1 60F7D6E2
-P 7650 2500
-F 0 "D1" H 7643 2245 50  0000 C CNN
-F 1 "Red LED" H 7643 2336 50  0000 C CNN
-F 2 "LED_SMD:LED_0603_1608Metric" H 7650 2500 50  0001 C CNN
-F 3 "~" H 7650 2500 50  0001 C CNN
-F 4 "C2286" H 7650 2500 50  0001 C CNN "LCSC"
-	1    7650 2500
-	-1   0    0    1
-$EndComp
-$Comp
-L Device:R R1
-U 1 1 60F8348E
-P 7350 2500
-F 0 "R1" V 7143 2500 50  0000 C CNN
-F 1 "5.1K" V 7234 2500 50  0000 C CNN
-F 2 "Resistor_SMD:R_0603_1608Metric" V 7280 2500 50  0001 C CNN
-F 3 "~" H 7350 2500 50  0001 C CNN
-F 4 "C23186" V 7350 2500 50  0001 C CNN "LCSC"
-	1    7350 2500
-	0    1    1    0
+P 7250 2450
+F 0 "D1" V 7250 2350 50  0000 C CNN
+F 1 "Red LED" V 7350 2250 50  0000 C CNN
+F 2 "LED_SMD:LED_0603_1608Metric" H 7250 2450 50  0001 C CNN
+F 3 "~" H 7250 2450 50  0001 C CNN
+F 4 "C2286" H 7250 2450 50  0001 C CNN "LCSC"
+	1    7250 2450
+	0    -1   -1   0
 $EndComp
 $Comp
@@
 F 0 "Q2" H 4455 3646 50  0000 L CNN
 F 1 "Q_NMOS_GSD 1Amp" H 4455 3555 50  0000 L CNN
-F 2 "Package_TO_SOT_SMD:SOT-23" H 4450 3700 50  0001 C CNN
+F 2 "Package_TO_SOT_SMD:SOT-723" H 4450 3700 50  0001 C CNN
 F 3 "~" H 4250 3600 50  0001 C CNN
-F 4 "C20917" H 4250 3600 50  0001 C CNN "LCSC"
+F 4 "C110712" H 4250 3600 50  0001 C CNN "LCSC"
 	1    4250 3600
 	-1   0    0    -1
@@
 F 0 "Q1" V 4400 3350 50  0000 C CNN
 F 1 "Q_PMOS_GSD, -3.6A 0.02R" V 4500 3050 50  0000 C CNN
-F 2 "Package_TO_SOT_SMD:SOT-23" H 4350 3300 50  0001 C CNN
+F 2 "Package_TO_SOT_SMD:SOT-883" H 4350 3300 50  0001 C CNN
 F 3 "~" H 4150 3200 50  0001 C CNN
-F 4 "C15127" V 4150 3200 50  0001 C CNN "LCSC"
+F 4 "C146297" V 4150 3200 50  0001 C CNN "LCSC"
 	1    4150 3200
 	0    -1   -1   0
@@
 F 0 "FB3" H 1950 5100 50  0000 L CNN
 F 1 "470 @ 100MHz" H 1400 4950 50  0001 L CNN
-F 2 "Inductor_SMD:L_0603_1608Metric" V 2130 5100 50  0001 C CNN
+F 2 "Inductor_SMD:L_0402_1005Metric" V 2130 5100 50  0001 C CNN
 F 3 "~" H 2200 5100 50  0001 C CNN
-F 4 "C97853" H 2200 5100 50  0001 C CNN "LCSC"
+F 4 "C333978" H 2200 5100 50  0001 C CNN "LCSC"
 	1    2200 5100
 	-1   0    0    1
@@
 F 0 "R13" H 7870 5596 50  0000 L CNN
 F 1 "2.7K" H 7870 5505 50  0000 L CNN
-F 2 "Resistor_SMD:R_0603_1608Metric" V 7730 5550 50  0001 C CNN
+F 2 "Resistor_SMD:R_0402_1005Metric" V 7730 5550 50  0001 C CNN
 F 3 "~" H 7800 5550 50  0001 C CNN
-F 4 "C13167" H 7800 5550 50  0001 C CNN "LCSC"
+F 4 "C25885" H 7800 5550 50  0001 C CNN "LCSC"
 	1    7800 5550
 	1    0    0    -1
@@
 F 0 "R12" H 7420 5596 50  0000 L CNN
 F 1 "2.7K" H 7420 5505 50  0000 L CNN
-F 2 "Resistor_SMD:R_0603_1608Metric" V 7280 5550 50  0001 C CNN
+F 2 "Resistor_SMD:R_0402_1005Metric" V 7280 5550 50  0001 C CNN
 F 3 "~" H 7350 5550 50  0001 C CNN
-F 4 "C13167" H 7350 5550 50  0001 C CNN "LCSC"
+F 4 "C25885" H 7350 5550 50  0001 C CNN "LCSC"
 	1    7350 5550
 	1    0    0    -1
@@
 Text GLabel 1100 1100 0    50   Input ~ 0
 NRST
-Text GLabel 1100 2000 0    50   Input ~ 0
-PC13
-$Comp
-L Device:LED D2
-U 1 1 60F6189C
-P 7650 2950
-F 0 "D2" H 7643 2695 50  0000 C CNN
-F 1 "Blue LED" H 7643 2786 50  0000 C CNN
-F 2 "LED_SMD:LED_0603_1608Metric" H 7650 2950 50  0001 C CNN
-F 3 "~" H 7650 2950 50  0001 C CNN
-F 4 "C72041" H 7650 2950 50  0001 C CNN "LCSC"
-	1    7650 2950
-	-1   0    0    1
-$EndComp
-$Comp
-L Device:R R4
-U 1 1 60F618A9
-P 7350 2950
-F 0 "R4" V 7143 2950 50  0000 C CNN
-F 1 "1.5K" V 7234 2950 50  0000 C CNN
-F 2 "Resistor_SMD:R_0603_1608Metric" V 7280 2950 50  0001 C CNN
-F 3 "~" H 7350 2950 50  0001 C CNN
-F 4 "C22843" V 7350 2950 50  0001 C CNN "LCSC"
-	1    7350 2950
-	0    1    1    0
-$EndComp
-Text GLabel 7800 2950 2    50   Input ~ 0
-PC13
-$Comp
-L power:+3.3V #PWR?
-U 1 1 60F618AF
-P 7200 2950
-AR Path="/60F56179/60F618AF" Ref="#PWR?"  Part="1"
-AR Path="/60F618AF" Ref="#PWR019"  Part="1"
-F 0 "#PWR019" H 7200 2800 50  0001 C CNN
-F 1 "+3.3V" H 7200 3100 50  0000 C CNN
-F 2 "" H 7200 2950 50  0001 C CNN
-F 3 "" H 7200 2950 50  0001 C CNN
-	1    7200 2950
-	0    -1   -1   0
-$EndComp
 Text Notes 8600 3050 0    50   ~ 0
 Reset
@@
 F 0 "FB2" H 3600 3100 50  0000 L CNN
 F 1 "470 @ 100MHz" H 3600 3050 50  0001 L CNN
-F 2 "Inductor_SMD:L_0603_1608Metric" V 3430 3100 50  0001 C CNN
+F 2 "Inductor_SMD:L_0402_1005Metric" V 3430 3100 50  0001 C CNN
 F 3 "~" H 3500 3100 50  0001 C CNN
-F 4 "C97853" H 3500 3100 50  0001 C CNN "LCSC"
+F 4 "C333978" H 3500 3100 50  0001 C CNN "LCSC"
 	1    3500 3100
 	0    -1   -1   0
@@
 	0    -1   1    0
 $EndComp
+Text GLabel 8850 5850 0    50   Input ~ 0
+SWDIO
+Text GLabel 8850 6050 0    50   Input ~ 0
+SWCLK
+NoConn ~ 1100 2000
+$Comp
+L Device:R_Small R1
+U 1 1 60F8348E
+P 7250 2650
+F 0 "R1" H 7150 2700 50  0000 C CNN
+F 1 "1K" H 7150 2600 50  0000 C CNN
+F 2 "Resistor_SMD:R_0402_1005Metric" V 7180 2650 50  0001 C CNN
+F 3 "~" H 7250 2650 50  0001 C CNN
+F 4 "C11702" V 7250 2650 50  0001 C CNN "LCSC"
+	1    7250 2650
+	-1   0    0    1
+$EndComp
+$Comp
+L power:GND #PWR?
+U 1 1 60F7E24C
+P 7250 2750
+AR Path="/60F56179/60F7E24C" Ref="#PWR?"  Part="1"
+AR Path="/60F7E24C" Ref="#PWR015"  Part="1"
+F 0 "#PWR015" H 7250 2500 50  0001 C CNN
+F 1 "GND" H 7250 2600 50  0000 C CNN
+F 2 "" H 7250 2750 50  0001 C CNN
+F 3 "" H 7250 2750 50  0001 C CNN
+	1    7250 2750
+	1    0    0    -1
+$EndComp
 $EndSCHEMATC
