File: Synapse.sch (KiCad schematic (older format))
At the start: 41 parts, among them J1 SWD, J2 I2C, SW1 SW_SPST, SW2 SW_SPST, U1 STM32F411CEUx, U2 SOT-553 LDO, U3 24LC256, Y1 24MHz 8pF, Y2 32.768K 7p

Commit message: PAUSED: Use `git resume` to continue working.
Parts:
- added C17: 470p, Capacitor_SMD:C_0402_1005Metric, symbol Device:C_Small
- C1, C8: value 1u -> 10u; LCSC C52923 -> C15525
- FB1, FB2: footprint Inductor_SMD:L_0402_1005Metric -> Inductor_SMD:L_0603_1608Metric; LCSC C185885 -> C114780
- U2: value SOT-553 LDO -> SOT-23-5 LDO (LM8805); footprint Package_TO_SOT_SMD:SOT-553 -> Package_TO_SOT_SMD:SOT-23-5; symbol Regulator_Linear:AMS1117-3.3 -> Regulator_Linear:SPX3819M5-L-3-3; LCSC C146430 -> C126077
Connections:
- net +3V3: now also U2.5 (OUT); no longer U2.2 (VO)
- net +5V: now also C1.2, U2.1 (IN); no longer C1.1, U2.3 (VI)
- net GND: now also C1.1, U2.2 (GND), C17.2; no longer C1.2, U2.1 (GND)
- new net: C17.1, U2.4 (BP)
Other:
- moved on the sheet: C1, C8
Changed lines of the file:
@@
 L power:+5V #PWR014
 U 1 1 60FBE829
-P 3350 1100
-F 0 "#PWR014" H 3350 950 50  0001 C CNN
-F 1 "+5V" H 3365 1273 50  0000 C CNN
-F 2 "" H 3350 1100 50  0001 C CNN
-F 3 "" H 3350 1100 50  0001 C CNN
-	1    3350 1100
-	1    0    0    -1
-$EndComp
-$Comp
-L power:GND #PWR015
-U 1 1 60FBEDF3
-P 3350 1300
-F 0 "#PWR015" H 3350 1050 50  0001 C CNN
-F 1 "GND" H 3355 1127 50  0000 C CNN
-F 2 "" H 3350 1300 50  0001 C CNN
-F 3 "" H 3350 1300 50  0001 C CNN
-	1    3350 1300
+P 3350 1000
+F 0 "#PWR014" H 3350 850 50  0001 C CNN
+F 1 "+5V" H 3365 1173 50  0000 C CNN
+F 2 "" H 3350 1000 50  0001 C CNN
+F 3 "" H 3350 1000 50  0001 C CNN
+	1    3350 1000
 	1    0    0    -1
 $EndComp
@@
 L power:+3.3V #PWR?
 U 1 1 60FC8BEA
-P 4250 1100
+P 4440 1000
 AR Path="/60F56179/60FC8BEA" Ref="#PWR?"  Part="1"
 AR Path="/60FC8BEA" Ref="#PWR029"  Part="1"
-F 0 "#PWR029" H 4250 950 50  0001 C CNN
-F 1 "+3.3V" H 4250 1250 50  0000 C CNN
-F 2 "" H 4250 1100 50  0001 C CNN
-F 3 "" H 4250 1100 50  0001 C CNN
-	1    4250 1100
+F 0 "#PWR029" H 4440 850 50  0001 C CNN
+F 1 "+3.3V" H 4440 1150 50  0000 C CNN
+F 2 "" H 4440 1000 50  0001 C CNN
+F 3 "" H 4440 1000 50  0001 C CNN
+	1    4440 1000
 	1    0    0    -1
 $EndComp
@@
 $EndComp
 $Comp
-L Regulator_Linear:AMS1117-3.3 U2
-U 1 1 60FBA365
-P 3800 1100
-F 0 "U2" H 3800 1342 50  0000 C CNN
-F 1 "SOT-553 LDO" H 3800 1251 50  0000 C CNN
-F 2 "Package_TO_SOT_SMD:SOT-553" H 3800 1300 50  0001 C CNN
-F 3 "" H 3900 850 50  0001 C CNN
-F 4 "C146430" H 3800 1100 50  0001 C CNN "LCSC"
-	1    3800 1100
-	1    0    0    -1
-$EndComp
-$Comp
 L Device:C_Small C?
 U 1 1 61066F3E
@@
 F 0 "FB2" V 3700 3050 50  0000 C CNN
 F 1 "470 @ 100MHz" V 3475 3100 50  0001 C CNN
-F 2 "Inductor_SMD:L_0402_1005Metric" H 3550 3100 50  0001 C CNN
+F 2 "Inductor_SMD:L_0603_1608Metric" H 3550 3100 50  0001 C CNN
 F 3 "~" H 3550 3100 50  0001 C CNN
-F 4 "C185885" H 3550 3100 50  0001 C CNN "LCSC"
+F 4 "C114780" H 3550 3100 50  0001 C CNN "LCSC"
 	1    3550 3100
 	0    -1   -1   0
@@
 F 0 "FB1" H 1650 6100 50  0000 L CNN
 F 1 "470 @ 100MHz" H 1100 5950 50  0001 L CNN
-F 2 "Inductor_SMD:L_0402_1005Metric" V 1830 6100 50  0001 C CNN
+F 2 "Inductor_SMD:L_0603_1608Metric" V 1830 6100 50  0001 C CNN
 F 3 "~" H 1900 6100 50  0001 C CNN
-F 4 "C185885" H 1900 6100 50  0001 C CNN "LCSC"
+F 4 "C114780" H 1900 6100 50  0001 C CNN "LCSC"
 	1    1900 6100
 	0    1    1    0
@@
 L Device:C_Small C?
 U 1 1 61341B47
-P 3350 1200
+P 3350 1100
 AR Path="/60F56179/61341B47" Ref="C?"  Part="1"
 AR Path="/61341B47" Ref="C1"  Part="1"
-F 0 "C1" H 3450 1250 50  0000 L CNN
-F 1 "1u" H 3450 1150 50  0000 L CNN
-F 2 "Capacitor_SMD:C_0402_1005Metric" H 3350 1200 50  0001 C CNN
-F 3 "~" H 3350 1200 50  0001 C CNN
-F 4 "C52923" H 3350 1200 50  0001 C CNN "LCSC"
-	1    3350 1200
-	1    0    0    -1
+F 0 "C1" H 3450 1050 50  0000 L CNN
+F 1 "10u" H 3450 1150 50  0000 L CNN
+F 2 "Capacitor_SMD:C_0402_1005Metric" H 3350 1100 50  0001 C CNN
+F 3 "~" H 3350 1100 50  0001 C CNN
+F 4 "C15525" H 3350 1100 50  0001 C CNN "LCSC"
+	1    3350 1100
+	-1   0    0    1
 $EndComp
 $Comp
 L Device:C_Small C?
 U 1 1 61347FB1
-P 4250 1200
+P 4440 1100
 AR Path="/60F56179/61347FB1" Ref="C?"  Part="1"
 AR Path="/61347FB1" Ref="C8"  Part="1"
-F 0 "C8" H 4350 1200 50  0000 L CNN
-F 1 "1u" H 4350 1100 50  0000 L CNN
-F 2 "Capacitor_SMD:C_0402_1005Metric" H 4250 1200 50  0001 C CNN
-F 3 "~" H 4250 1200 50  0001 C CNN
-F 4 "C52923" H 4250 1200 50  0001 C CNN "LCSC"
-	1    4250 1200
-	1    0    0    -1
-$EndComp
-$Comp
-L power:GND #PWR030
-U 1 1 61348DC9
-P 4250 1300
-F 0 "#PWR030" H 4250 1050 50  0001 C CNN
-F 1 "GND" H 4255 1127 50  0000 C CNN
-F 2 "" H 4250 1300 50  0001 C CNN
-F 3 "" H 4250 1300 50  0001 C CNN
-	1    4250 1300
-	1    0    0    -1
-$EndComp
-Wire Wire Line
-	4100 1100 4250 1100
-Connection ~ 4250 1100
-Wire Wire Line
-	3350 1100 3500 1100
-Connection ~ 3350 1100
+F 0 "C8" H 4550 1150 50  0000 L CNN
+F 1 "10u" H 4550 1050 50  0000 L CNN
+F 2 "Capacitor_SMD:C_0402_1005Metric" H 4440 1100 50  0001 C CNN
+F 3 "~" H 4440 1100 50  0001 C CNN
+F 4 "C15525" H 4440 1100 50  0001 C CNN "LCSC"
+	1    4440 1100
+	1    0    0    -1
+$EndComp
+Connection ~ 4440 1000
+Wire Wire Line
+	3350 1000 3500 1000
 Text Notes 3250 2850 0    50   ~ 0
 Analog power filtering\n
@@
 I2C1_SDA
 NoConn ~ 1200 3600
+$Comp
+L Regulator_Linear:SPX3819M5-L-3-3 U2
+U 1 1 60FBA365
+P 3800 1100
+F 0 "U2" H 3800 1342 50  0000 C CNN
+F 1 "SOT-23-5 LDO (LM8805)" H 4430 1440 50  0000 C CNN
+F 2 "Package_TO_SOT_SMD:SOT-23-5" H 3800 1300 50  0001 C CNN
+F 3 "" H 3900 850 50  0001 C CNN
+F 4 "C126077" H 3800 1100 50  0001 C CNN "LCSC"
+	1    3800 1100
+	1    0    0    -1
+$EndComp
+Connection ~ 3350 1000
+$Comp
+L Device:C_Small C?
+U 1 1 610733A3
+P 4100 1200
+AR Path="/60F56179/610733A3" Ref="C?"  Part="1"
+AR Path="/610733A3" Ref="C17"  Part="1"
+F 0 "C17" H 4200 1250 50  0000 L CNN
+F 1 "470p" H 4200 1150 50  0000 L CNN
+F 2 "Capacitor_SMD:C_0402_1005Metric" H 4100 1200 50  0001 C CNN
+F 3 "~" H 4100 1200 50  0001 C CNN
+F 4 "C1537" H 4100 1200 50  0001 C CNN "LCSC"
+	1    4100 1200
+	1    0    0    -1
+$EndComp
+Wire Wire Line
+	4100 1000 4440 1000
+Wire Wire Line
+	4100 1400 4100 1300
+Wire Wire Line
+	3800 1400 4100 1400
+Connection ~ 4100 1400
+Wire Wire Line
+	4100 1400 4440 1400
+Wire Wire Line
+	3800 1400 3350 1400
+Wire Wire Line
+	3350 1400 3350 1200
+Connection ~ 3800 1400
+Wire Wire Line
+	4440 1200 4440 1400
 $EndSCHEMATC

Commit message: PAUSED: Use `git resume` to continue working.
Parts:
- removed C8: 10u, Capacitor_SMD:C_0402_1005Metric, symbol Device:C_Small
- removed J2: I2C, Common:TestPoint_Pads_4x2.54_D1.5mm, symbol Connector_Generic:Conn_01x04
- removed R8: 10k, Resistor_SMD:R_0402_1005Metric, symbol Device:R_Small
- removed SW1: SW_SPST, Button_Switch_SMD:SW_SPST_B3U-1000P, symbol Switch:SW_Push
- C1: value 10u -> 1u; LCSC C15525 -> C52923
- C17: value 470p -> 1u; LCSC C1537 -> C52923
- J1: footprint Common:TestPoint_Pads_4x2.54_D1.5mm -> Common:TestPoint_Pads_5x2.54_D1.5mm; symbol Connector_Generic:Conn_01x04 -> Connector_Generic:Conn_01x05
- U2: value SOT-23-5 LDO (LM8805) -> SOT-23-3L LDO 200mA; footprint Package_TO_SOT_SMD:SOT-23-5 -> Package_TO_SOT_SMD:SOT-23; symbol Regulator_Linear:SPX3819M5-L-3-3 -> Regulator_Linear:MCP1700-3302E_SOT23; LCSC C126077 -> C5446
Connections:
- net +3V3: now also C17.1, J1.5 (Pin_5), U2.2 (VO); no longer J1.4 (Pin_4), U2.5 (OUT)
- net +5V: now also C1.1, U2.3 (VI); no longer C1.2, U2.1 (IN)
- net GND: now also C1.2, U2.1 (GND); no longer C1.1, U2.2 (GND)
- net NRST: now also J1.2 (Pin_2)
- net SWCLK: now also J1.3 (Pin_3); no longer J1.2 (Pin_2)
- net SWDIO: now also J1.4 (Pin_4); no longer J1.3 (Pin_3)
Other:
- moved on the sheet: C1, C16
Changed lines of the file:
@@
 L power:+5V #PWR014
 U 1 1 60FBE829
-P 3350 1000
-F 0 "#PWR014" H 3350 850 50  0001 C CNN
-F 1 "+5V" H 3365 1173 50  0000 C CNN
-F 2 "" H 3350 1000 50  0001 C CNN
-F 3 "" H 3350 1000 50  0001 C CNN
-	1    3350 1000
+P 3350 1100
+F 0 "#PWR014" H 3350 950 50  0001 C CNN
+F 1 "+5V" H 3365 1273 50  0000 C CNN
+F 2 "" H 3350 1100 50  0001 C CNN
+F 3 "" H 3350 1100 50  0001 C CNN
+	1    3350 1100
 	1    0    0    -1
 $EndComp
@@
 L power:+3.3V #PWR?
 U 1 1 60FC8BEA
-P 4440 1000
+P 4250 1100
 AR Path="/60F56179/60FC8BEA" Ref="#PWR?"  Part="1"
 AR Path="/60FC8BEA" Ref="#PWR029"  Part="1"
-F 0 "#PWR029" H 4440 850 50  0001 C CNN
-F 1 "+3.3V" H 4440 1150 50  0000 C CNN
-F 2 "" H 4440 1000 50  0001 C CNN
-F 3 "" H 4440 1000 50  0001 C CNN
-	1    4440 1000
+F 0 "#PWR029" H 4250 950 50  0001 C CNN
+F 1 "+3.3V" H 4250 1250 50  0000 C CNN
+F 2 "" H 4250 1100 50  0001 C CNN
+F 3 "" H 4250 1100 50  0001 C CNN
+	1    4250 1100
 	1    0    0    -1
 $EndComp
@@
 Wire Wire Line
 	3750 3300 4050 3300
-$Comp
-L Device:C_Small C?
-U 1 1 61341B47
-P 3350 1100
-AR Path="/60F56179/61341B47" Ref="C?"  Part="1"
-AR Path="/61341B47" Ref="C1"  Part="1"
-F 0 "C1" H 3450 1050 50  0000 L CNN
-F 1 "10u" H 3450 1150 50  0000 L CNN
-F 2 "Capacitor_SMD:C_0402_1005Metric" H 3350 1100 50  0001 C CNN
-F 3 "~" H 3350 1100 50  0001 C CNN
-F 4 "C15525" H 3350 1100 50  0001 C CNN "LCSC"
-	1    3350 1100
-	-1   0    0    1
-$EndComp
-$Comp
-L Device:C_Small C?
-U 1 1 61347FB1
-P 4440 1100
-AR Path="/60F56179/61347FB1" Ref="C?"  Part="1"
-AR Path="/61347FB1" Ref="C8"  Part="1"
-F 0 "C8" H 4550 1150 50  0000 L CNN
-F 1 "10u" H 4550 1050 50  0000 L CNN
-F 2 "Capacitor_SMD:C_0402_1005Metric" H 4440 1100 50  0001 C CNN
-F 3 "~" H 4440 1100 50  0001 C CNN
-F 4 "C15525" H 4440 1100 50  0001 C CNN "LCSC"
-	1    4440 1100
-	1    0    0    -1
-$EndComp
-Connection ~ 4440 1000
-Wire Wire Line
-	3350 1000 3500 1000
 Text Notes 3250 2850 0    50   ~ 0
 Analog power filtering\n
@@
 	3700 5050 3700 4950
 $Comp
-L power:GND #PWR?
-U 1 1 61097B2D
-P 9400 2900
-AR Path="/60F56179/61097B2D" Ref="#PWR?"  Part="1"
-AR Path="/61097B2D" Ref="#PWR049"  Part="1"
-F 0 "#PWR049" H 9400 2650 50  0001 C CNN
-F 1 "GND" H 9400 2750 50  0000 C CNN
-F 2 "" H 9400 2900 50  0001 C CNN
-F 3 "" H 9400 2900 50  0001 C CNN
-	1    9400 2900
-	1    0    0    -1
-$EndComp
-Wire Wire Line
-	9400 2900 9400 2800
-Text GLabel 9400 2500 1    50   Input ~ 0
-BOOT1
-Wire Wire Line
-	9400 2500 9400 2600
-$Comp
 L Device:R_Small R?
 U 1 1 60FB29E6
@@
 Reset
 $Comp
-L power:+3.3V #PWR?
-U 1 1 613B41A1
-P 8850 3750
-AR Path="/60F56179/613B41A1" Ref="#PWR?"  Part="1"
-AR Path="/613B41A1" Ref="#PWR046"  Part="1"
-F 0 "#PWR046" H 8850 3600 50  0001 C CNN
-F 1 "+3.3V" H 8850 3900 50  0000 C CNN
-F 2 "" H 8850 3750 50  0001 C CNN
-F 3 "" H 8850 3750 50  0001 C CNN
-	1    8850 3750
-	1    0    0    -1
-$EndComp
-$Comp
 L power:GND #PWR?
 U 1 1 613B41AC
-P 8750 4650
+P 8750 4150
 AR Path="/60F56179/613B41AC" Ref="#PWR?"  Part="1"
 AR Path="/613B41AC" Ref="#PWR045"  Part="1"
-F 0 "#PWR045" H 8750 4400 50  0001 C CNN
-F 1 "GND" H 8750 4500 50  0000 C CNN
-F 2 "" H 8750 4650 50  0001 C CNN
-F 3 "" H 8750 4650 50  0001 C CNN
-	1    8750 4650
-	1    0    0    -1
-$EndComp
-Wire Wire Line
-	8850 4600 8750 4600
-Connection ~ 8750 4600
-Wire Wire Line
-	8750 4600 8750 4650
-Wire Wire Line
-	8750 4600 8650 4600
-Wire Wire Line
-	8650 4600 8650 4500
-$Comp
-L Device:R_Small R?
-U 1 1 613B41C0
-P 8850 3850
-AR Path="/60F56179/613B41C0" Ref="R?"  Part="1"
-AR Path="/613B41C0" Ref="R8"  Part="1"
-F 0 "R8" V 8775 3850 50  0000 C CNN
-F 1 "10k" V 8925 3850 50  0000 C CNN
-F 2 "Resistor_SMD:R_0402_1005Metric" H 8850 3850 50  0001 C CNN
-F 3 "~" H 8850 3850 50  0001 C CNN
-F 4 "C25744" H 8850 3850 50  0001 C CNN "LCSC"
-	1    8850 3850
-	-1   0    0    1
+F 0 "#PWR045" H 8750 3900 50  0001 C CNN
+F 1 "GND" H 8750 4000 50  0000 C CNN
+F 2 "" H 8750 4150 50  0001 C CNN
+F 3 "" H 8750 4150 50  0001 C CNN
+	1    8750 4150
+	1    0    0    -1
 $EndComp
 $Comp
 L Device:C_Small C?
 U 1 1 613B41C7
-P 8650 4400
+P 8750 4050
 AR Path="/60F56179/613B41C7" Ref="C?"  Part="1"
 AR Path="/613B41C7" Ref="C16"  Part="1"
-F 0 "C16" H 8750 4450 50  0000 L CNN
-F 1 "100n" H 8750 4350 50  0000 L CNN
-F 2 "Capacitor_SMD:C_0402_1005Metric" H 8650 4400 50  0001 C CNN
-F 3 "~" H 8650 4400 50  0001 C CNN
-F 4 "C1525" H 8650 4400 50  0001 C CNN "LCSC"
-	1    8650 4400
+F 0 "C16" H 8850 4100 50  0000 L CNN
+F 1 "100n" H 8850 4000 50  0000 L CNN
+F 2 "Capacitor_SMD:C_0402_1005Metric" H 8750 4050 50  0001 C CNN
+F 3 "~" H 8750 4050 50  0001 C CNN
+F 4 "C1525" H 8750 4050 50  0001 C CNN "LCSC"
+	1    8750 4050
 	-1   0    0    1
 $EndComp
-$Comp
-L Switch:SW_Push SW1
-U 1 1 613B41B9
-P 8850 4400
-F 0 "SW1" H 8850 4685 50  0000 C CNN
-F 1 "SW_SPST" H 8850 4594 50  0000 C CNN
-F 2 "Button_Switch_SMD:SW_SPST_B3U-1000P" H 8850 4600 50  0001 C CNN
-F 3 "~" H 8850 4600 50  0001 C CNN
-F 4 "C231329" H 8850 4400 50  0001 C CNN "LCSC"
-	1    8850 4400
-	0    1    1    0
-$EndComp
-Text GLabel 8600 4050 0    50   Input ~ 0
+Text GLabel 8750 3950 1    50   Input ~ 0
 NRST
-Wire Wire Line
-	8650 4300 8650 4200
-Wire Wire Line
-	8650 4200 8850 4200
-Wire Wire Line
-	8850 3950 8850 4050
-Connection ~ 8850 4200
-Wire Wire Line
-	8600 4050 8850 4050
-Connection ~ 8850 4050
-Wire Wire Line
-	8850 4050 8850 4200
 Text GLabel 7200 5450 2    50   Input ~ 0
 SWCLK
@@
 $EndComp
 $Comp
-L Connector_Generic:Conn_01x04 J1
+L Connector_Generic:Conn_01x05 J1
 U 1 1 61003A04
 P 7000 5450
 F 0 "J1" H 7100 5450 50  0000 L CNN
 F 1 "SWD" H 7100 5350 50  0000 L CNN
-F 2 "Common:TestPoint_Pads_4x2.54_D1.5mm" H 7000 5450 50  0001 C CNN
+F 2 "Common:TestPoint_Pads_5x2.54_D1.5mm" H 7000 5450 50  0001 C CNN
 F 3 "~" H 7000 5450 50  0001 C CNN
 	1    7000 5450
@@
 L power:GND #PWR042
 U 1 1 60F704A2
-P 7200 5550
-F 0 "#PWR042" H 7200 5300 50  0001 C CNN
-F 1 "GND" V 7200 5350 50  0000 C CNN
-F 2 "" H 7200 5550 50  0001 C CNN
-F 3 "" H 7200 5550 50  0001 C CNN
-	1    7200 5550
+P 7200 5650
+F 0 "#PWR042" H 7200 5400 50  0001 C CNN
+F 1 "GND" V 7200 5450 50  0000 C CNN
+F 2 "" H 7200 5650 50  0001 C CNN
+F 3 "" H 7200 5650 50  0001 C CNN
+	1    7200 5650
 	0    -1   1    0
 $EndComp
-$Comp
-L Connector_Generic:Conn_01x04 J2
-U 1 1 610BAE66
-P 7900 5450
-F 0 "J2" V 8000 5300 50  0000 L CNN
-F 1 "I2C" V 8000 5400 50  0000 L CNN
-F 2 "Common:TestPoint_Pads_4x2.54_D1.5mm" H 7900 5450 50  0001 C CNN
-F 3 "~" H 7900 5450 50  0001 C CNN
-	1    7900 5450
-	-1   0    0    1
-$EndComp
-$Comp
-L power:+5V #PWR?
-U 1 1 610F4CC7
-P 8100 5250
-AR Path="/60F56179/610F4CC7" Ref="#PWR?"  Part="1"
-AR Path="/610F4CC7" Ref="#PWR043"  Part="1"
-F 0 "#PWR043" H 8100 5100 50  0001 C CNN
-F 1 "+5V" V 8100 5450 50  0000 C CNN
-F 2 "" H 8100 5250 50  0001 C CNN
-F 3 "" H 8100 5250 50  0001 C CNN
-	1    8100 5250
-	0    1    -1   0
-$EndComp
-$Comp
-L power:GND #PWR044
-U 1 1 610EF04D
-P 8100 5550
-F 0 "#PWR044" H 8100 5300 50  0001 C CNN
-F 1 "GND" V 8100 5350 50  0000 C CNN
-F 2 "" H 8100 5550 50  0001 C CNN
-F 3 "" H 8100 5550 50  0001 C CNN
-	1    8100 5550
-	0    -1   -1   0
-$EndComp
-Text GLabel 8100 5450 2    50   Input ~ 0
-I2C1_SCL
-Text GLabel 8100 5350 2    50   Input ~ 0
-I2C1_SDA
 $Comp
 L power:+5V #PWR035
@@
 NoConn ~ 1200 3600
 $Comp
-L Regulator_Linear:SPX3819M5-L-3-3 U2
+L Regulator_Linear:MCP1700-3302E_SOT23 U2
 U 1 1 60FBA365
 P 3800 1100
 F 0 "U2" H 3800 1342 50  0000 C CNN
-F 1 "SOT-23-5 LDO (LM8805)" H 4430 1440 50  0000 C CNN
-F 2 "Package_TO_SOT_SMD:SOT-23-5" H 3800 1300 50  0001 C CNN
+F 1 "SOT-23-3L LDO 200mA" H 4430 1440 50  0000 C CNN
+F 2 "Package_TO_SOT_SMD:SOT-23" H 3800 1300 50  0001 C CNN
 F 3 "" H 3900 850 50  0001 C CNN
-F 4 "C126077" H 3800 1100 50  0001 C CNN "LCSC"
+F 4 "C5446" H 3800 1100 50  0001 C CNN "LCSC"
 	1    3800 1100
 	1    0    0    -1
 $EndComp
-Connection ~ 3350 1000
 $Comp
 L Device:C_Small C?
@@
 AR Path="/610733A3" Ref="C17"  Part="1"
 F 0 "C17" H 4200 1250 50  0000 L CNN
-F 1 "470p" H 4200 1150 50  0000 L CNN
+F 1 "1u" H 4200 1150 50  0000 L CNN
 F 2 "Capacitor_SMD:C_0402_1005Metric" H 4100 1200 50  0001 C CNN
 F 3 "~" H 4100 1200 50  0001 C CNN
-F 4 "C1537" H 4100 1200 50  0001 C CNN "LCSC"
+F 4 "C52923" H 4100 1200 50  0001 C CNN "LCSC"
 	1    4100 1200
 	1    0    0    -1
 $EndComp
-Wire Wire Line
-	4100 1000 4440 1000
-Wire Wire Line
-	4100 1400 4100 1300
-Wire Wire Line
-	3800 1400 4100 1400
-Connection ~ 4100 1400
-Wire Wire Line
-	4100 1400 4440 1400
-Wire Wire Line
-	3800 1400 3350 1400
-Wire Wire Line
-	3350 1400 3350 1200
+Text GLabel 7200 5550 2    50   Input ~ 0
+NRST
+$Comp
+L power:GND #PWR?
+U 1 1 61097B2D
+P 9400 2900
+AR Path="/60F56179/61097B2D" Ref="#PWR?"  Part="1"
+AR Path="/61097B2D" Ref="#PWR049"  Part="1"
+F 0 "#PWR049" H 9400 2650 50  0001 C CNN
+F 1 "GND" H 9400 2750 50  0000 C CNN
+F 2 "" H 9400 2900 50  0001 C CNN
+F 3 "" H 9400 2900 50  0001 C CNN
+	1    9400 2900
+	1    0    0    -1
+$EndComp
+Wire Wire Line
+	9400 2900 9400 2800
+Text GLabel 9400 2500 1    50   Input ~ 0
+BOOT1
+Wire Wire Line
+	9400 2500 9400 2600
+Wire Wire Line
+	4250 1100 4100 1100
+Connection ~ 4100 1100
+Wire Wire Line
+	4100 1300 4100 1400
+Wire Wire Line
+	4100 1400 3800 1400
 Connection ~ 3800 1400
-Wire Wire Line
-	4440 1200 4440 1400
+$Comp
+L Device:C_Small C?
+U 1 1 61341B47
+P 3500 1200
+AR Path="/60F56179/61341B47" Ref="C?"  Part="1"
+AR Path="/61341B47" Ref="C1"  Part="1"
+F 0 "C1" H 3600 1150 50  0000 L CNN
+F 1 "1u" H 3600 1250 50  0000 L CNN
+F 2 "Capacitor_SMD:C_0402_1005Metric" H 3500 1200 50  0001 C CNN
+F 3 "~" H 3500 1200 50  0001 C CNN
+F 4 "C52923" H 3500 1200 50  0001 C CNN "LCSC"
+	1    3500 1200
+	-1   0    0    -1
+$EndComp
+Wire Wire Line
+	3500 1300 3500 1400
+Wire Wire Line
+	3500 1400 3800 1400
+Connection ~ 3500 1100
+Wire Wire Line
+	3350 1100 3500 1100
 $EndSCHEMATC

Commit message: Final form
Parts:
- added FB2: 470 @ 100MHz, Inductor_SMD:L_0603_1608Metric, symbol Device:Ferrite_Bead_Small
- FB1: renamed from FB2; LCSC C114780 -> C356977
- FB3: renamed from FB1; LCSC C114780 -> C356977
- renumbered C15 to C10, C5 to C11, C6 to C12, C12 to C13, C3 to C15, C17 to C2, C10 to C3, C2 to C4, C4 to C5, C7 to C6, C9 to C7, C11 to C8, C13 to C9, R10 to R1, R9 to R2, R6 to R3, R3 to R4, R1 to R6, R4 to R7, R7 to R8, R2 to R9, SW2 to SW1, U2 to U1, U3 to U2, U1 to U3
Connections:
- net +5V: now also FB2.1
- net NRST: now also J1.4 (Pin_4); no longer J1.2 (Pin_2)
- net SWDIO: now also J1.2 (Pin_2); no longer J1.4 (Pin_4)
- net at FB3.2, USB1.A4 (VBUS), USB1.A9 (VBUS)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: now also FB2.2
Other:
- note added: "One FB per pin"
