File: Synapse.kicad_pcb (KiCad board)
At the start: 2 copper layers, 89.5 x 74.9 mm, 32 parts, among them SW1 SW_SPST, SW2 SW_SPST, U4 STM32F411CEUx, U5 AMS1117-3.3, Y1 25MHz 9pF, Y2 32.768K 7pF

Commit message: PAUSED: Use `git resume` to continue working.
Parts:
- removed C17, C18: 8pF, Capacitor_SMD:C_0402_1005Metric
- removed C19, C20: 4pF, Capacitor_SMD:C_0402_1005Metric
- removed C21, C23, C28: 4u7, Capacitor_SMD:C_0603_1608Metric
- removed C22, C25, C27, C29, C31, C32, C33: 100n, Capacitor_SMD:C_0402_1005Metric
- removed C24: 1u, Capacitor_SMD:C_0402_1005Metric
- removed C26, C30: 10n, Capacitor_SMD:C_0402_1005Metric
- removed L3: 39n, Inductor_SMD:L_0402_1005Metric
- removed R12, R8: 5.1K, Resistor_SMD:R_0805_2012Metric
- removed R13, R14, R15: 10k, Resistor_SMD:R_0402_1005Metric
- removed SW1, SW2: SW_SPST, Button_Switch_SMD:SW_SPST_PTS645
- removed U4: STM32F411CEUx, Package_DFN_QFN:QFN-48-1EP_7x7mm_P0.5mm_EP5.6x5.6mm
- removed U5: AMS1117-3.3, Package_TO_SOT_SMD:SOT-223-3_TabPin2
- removed USB1, USB2, USB3: USB_C_Receptacle_USB2.0, Connector_USB:USB_C_Receptacle_HRO_TYPE-C-31-M-12
- removed Y1: 25MHz 9pF, Crystal:Crystal_SMD_2520-4Pin_2.5x2.0mm
- removed Y2: 32.768K 7pF, Crystal:Crystal_SMD_2012-2Pin_2.0x1.2mm
Routing:
- net GND: track 26.5 -> 0.00 mm, vias 4 -> 0
- net Net-(R12-Pad2): track 7.80 -> 0.00 mm
- net Net-(R8-Pad2): track 7.76 -> 0.00 mm
- net +3V3: track 3.06 -> 0.00 mm
- net +5V: track 3.04 -> 0.00 mm
- net PB2: track 2.14 -> 0.00 mm
- removed copper zone on F.Cu, net +3V3
- removed copper zone on B.Cu, net GND
Other:
- board outline removed

Commit message: PAUSED: Use `git resume` to continue working.
Parts:
- added C1: 100n, Capacitor_SMD:C_0402_1005Metric, F.Cu at (0.00, 0.00)
- added C10: 4p, Capacitor_SMD:C_0402_1005Metric, F.Cu at (9.29, -11.2)
- added C11: 1u, Capacitor_SMD:C_0402_1005Metric, F.Cu at (-6.57, 4.06)
- added C12: 100n, Capacitor_SMD:C_0402_1005Metric, F.Cu at (5.62, -8.70)
- added C13: 100n, Capacitor_SMD:C_0402_1005Metric, F.Cu at (0.87, -3.96)
- added C14: 100pF ceramic, 100v, 10%, Capacitor_SMD:C_0805_2012Metric, F.Cu at (-38.4, 5.65)
- added C15: 4u7, Capacitor_SMD:C_0603_1608Metric, F.Cu at (-1.47, -8.71)
- added C16: 4u7, Capacitor_SMD:C_0603_1608Metric, F.Cu at (8.15, -15.4)
- added C17: 10n, Capacitor_SMD:C_0402_1005Metric, F.Cu at (-6.57, 2.09)
- added C18: 100n, Capacitor_SMD:C_0402_1005Metric, F.Cu at (9.29, -13.1)
- added C19: 100n, Capacitor_SMD:C_0402_1005Metric, F.Cu at (-2.87, -0.42)
- added C2: 4u7, Capacitor_SMD:C_0603_1608Metric, F.Cu at (2.94, -11.7)
- added C3: 100n, Capacitor_SMD:C_0402_1005Metric, F.Cu at (-3.70, 4.06)
- added C4: 100n, Capacitor_SMD:C_0402_1005Metric, F.Cu at (8.49, -8.70)
- added C5: 100n, Capacitor_SMD:C_0402_1005Metric, F.Cu at (3.74, -4.14)
- added C6: 100n, Capacitor_SMD:C_0402_1005Metric, F.Cu at (0.00, -1.97)
- added C7: 8p, Capacitor_SMD:C_0402_1005Metric, F.Cu at (4.88, -6.13)
- added C8: 8p, Capacitor_SMD:C_0402_1005Metric, F.Cu at (-7.67, 6.14)
- added C9: 4p, Capacitor_SMD:C_0402_1005Metric, F.Cu at (-3.70, 2.09)
- added D1: RED LED, LED_SMD:LED_0603_1608Metric, F.Cu at (-18.4, 5.80)
- added D2: BLUE LED, LED_SMD:LED_0603_1608Metric, F.Cu at (-14.0, 3.94)
- added FB1: 120Ω @ 100MHz, Inductor_SMD:L_0603_1608Metric, F.Cu at (-1.47, -6.20)
- added FB2: 120Ω @ 100MHz, Inductor_SMD:L_0603_1608Metric, F.Cu at (-14.4, 6.49)
- added J1: Conn_01x04_Female, Connector_PinHeader_2.54mm:PinHeader_1x04_P2.54mm_Vertical, F.Cu at (-22.1, -18.8)
- added L1: 39n, Inductor_SMD:L_0402_1005Metric, F.Cu at (6.40, -10.7)
- added Q1: Q_PMOS_GSD, -3.6A 0.02R, Package_TO_SOT_SMD:SOT-23, F.Cu at (-26.7, -4.05)
- added Q2: Q_NMOS_GSD 1Amp, Package_TO_SOT_SMD:SOT-23, F.Cu at (3.96, -18.9)
- added R1: 5.1K, Resistor_SMD:R_0603_1608Metric, F.Cu at (-10.0, 3.90)
- added R10: 200k, Resistor_SMD:R_0805_2012Metric, F.Cu at (8.39, -19.7)
- added R11: 5.1K, Resistor_SMD:R_0402_1005Metric, F.Cu at (-10.6, 6.15)
- added R12: 2.7K, Resistor_SMD:R_0805_2012Metric, F.Cu at (-26.7, -0.30)
- added R13: 2.7K, Resistor_SMD:R_0805_2012Metric, F.Cu at (-34.0, 5.62)
- added R2: 10k, Resistor_SMD:R_0402_1005Metric, F.Cu at (6.40, -12.7)
- added R3: 10k, Resistor_SMD:R_0402_1005Metric, F.Cu at (-6.66, -11.9)
- added R4: 1.5K, Resistor_SMD:R_0603_1608Metric, F.Cu at (-6.31, -0.15)
- added R5: 10k, Resistor_SMD:R_0402_1005Metric, F.Cu at (-2.02, -3.95)
- added R6: 10k. 125mW. 5%., Resistor_SMD:R_0805_2012Metric, F.Cu at (-1.27, -11.4)
- added R7: 10k. 125mW. 5%., Resistor_SMD:R_0805_2012Metric, F.Cu at (-18.3, 3.03)
- added R8: 5.1K, Resistor_SMD:R_0402_1005Metric, F.Cu at (1.99, -6.12)
- added R9: 200k, Resistor_SMD:R_0805_2012Metric, F.Cu at (3.94, -15.1)
- added SW1: SW_SPST, Common:K2-1102SP-C4SC-04, F.Cu at (-32.4, -9.88)
- added SW2: SW_SPST, Common:K2-1102SP-C4SC-04, F.Cu at (-32.4, -17.3)
- added U1: STM32F411CEUx, Package_DFN_QFN:QFN-48-1EP_7x7mm_P0.5mm_EP5.6x5.6mm, F.Cu at (-8.12, -6.05)
- added U2: AMS1117-3.3, Package_TO_SOT_SMD:SOT-223-3_TabPin2, F.Cu at (-3.19, -17.0)
- added U3: 24LC256, Package_SO:SOIC-8_3.9x4.9mm_P1.27mm, F.Cu at (-24.7, 4.78)
- added USB1: USB_C_Receptacle_USB2.0, Connector_USB:USB_C_Receptacle_HRO_TYPE-C-31-M-12, F.Cu at (-18.6, -3.12)
- added USB2: USB_C_Receptacle_USB2.0, Connector_USB:USB_C_Receptacle_HRO_TYPE-C-31-M-12, F.Cu at (-14.0, -15.4)
- added USB3: USB_C_Receptacle_USB2.0, Connector_USB:USB_C_Receptacle_HRO_TYPE-C-31-M-12, F.Cu at (-34.8, -0.53)
- added Y1: 25MHz 9pF, Crystal:Crystal_SMD_2520-4Pin_2.5x2.0mm, F.Cu at (-10.5, 0.62)
- added Y2: 32.768K 7pF, Crystal:Crystal_SMD_2012-2Pin_2.0x1.2mm, F.Cu at (2.36, -8.54)

Commit message: PAUSED: Use `git resume` to continue working.
Parts:
- removed L1: 39n, Inductor_SMD:L_0402_1005Metric
- added FB3: 470 @ 100MHz, Inductor_SMD:L_0603_1608Metric, F.Cu at (6.35, -11.4)
- added R14: 2.7K, Resistor_SMD:R_0603_1608Metric, F.Cu at (-6.35, -8.89)
- C10, C9: value 4p -> 15p
- C14: value 100pF ceramic, 100v, 10% -> 100p; footprint Capacitor_SMD:C_0805_2012Metric -> Capacitor_SMD:C_0402_1005Metric
- C7, C8: value 8p -> 15p
- D1: value RED LED -> Red LED
- D2: value BLUE LED -> Blue LED
- FB1, FB2: value 120Ω @ 100MHz -> 470 @ 100MHz
- R1: value 5.1K -> 330; footprint Resistor_SMD:R_0603_1608Metric -> Resistor_SMD:R_0402_1005Metric
- R10: footprint Resistor_SMD:R_0805_2012Metric -> Resistor_SMD:R_0402_1005Metric
- R11: value 5.1K -> 200k
- R12: value 2.7K -> 5.1K; footprint Resistor_SMD:R_0805_2012Metric -> Resistor_SMD:R_0402_1005Metric
- R13: footprint Resistor_SMD:R_0805_2012Metric -> Resistor_SMD:R_0603_1608Metric
- R2: value 10k -> 5.1K; footprint Resistor_SMD:R_0402_1005Metric -> Resistor_SMD:R_0603_1608Metric
- R4: value 1.5K -> 10k; footprint Resistor_SMD:R_0603_1608Metric -> Resistor_SMD:R_0402_1005Metric
- R5: value 10k -> 1.5K; footprint Resistor_SMD:R_0402_1005Metric -> Resistor_SMD:R_0603_1608Metric
- R6, R7: value 10k. 125mW. 5%. -> 10k; footprint Resistor_SMD:R_0805_2012Metric -> Resistor_SMD:R_0402_1005Metric
- R8: value 5.1K -> 10k
- R9: value 200k -> 5.1K; footprint Resistor_SMD:R_0805_2012Metric -> Resistor_SMD:R_0402_1005Metric
- Y1: value 25MHz 9pF -> 25MHz 12pF; footprint Crystal:Crystal_SMD_2520-4Pin_2.5x2.0mm -> Crystal:Crystal_SMD_3225-4Pin_3.2x2.5mm
- Y2: value 32.768K 7pF -> 32.768K 12.5p; footprint Crystal:Crystal_SMD_2012-2Pin_2.0x1.2mm -> Crystal:Crystal_SMD_3215-2Pin_3.2x1.5mm
- moved R10 91.7 mm to (-47.0, 53.3)
- moved USB3 87.9 mm to (30.5, 58.4)
- moved J1 80.4 mm to (-5.08, 59.7), turned to 90 degrees
- moved USB2 73.6 mm to (-36.8, 54.6)
- moved R11 71.4 mm to (39.4, 57.1)
- moved Q2 71.1 mm to (-15.2, 49.5)
- moved D1 69.6 mm to (49.5, -9.50)
- moved D2 68.9 mm to (53.5, -9.50)
- moved SW1 63.1 mm to (30.5, -3.81)
- moved SW2 62.9 mm to (30.5, -15.2)
- moved R8 62.7 mm to (-17.8, 53.3)
- moved R5 61.0 mm to (58.6, -10.9)
- moved C16 58.3 mm to (45.7, 29.2)
- moved C17 54.2 mm to (45.7, 16.5)
- moved C14 54.2 mm to (-12.7, 53.3)
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Connections:
- C8 pad 1: HSE_IN -> Net-(C8-Pad1)
- FB1 pad 1: SIDE_POWER -> +3V3
- FB1 pad 2: Net-(C14-Pad1) -> +3.3VA
- FB2 pad 1: Net-(FB2-Pad1) -> SIDE_POWER
- FB2 pad 2: +5V -> Net-(C14-Pad1)
- R1 pad 1: Net-(D1-Pad2) -> HSE_IN
- R1 pad 2: +3V3 -> Net-(C8-Pad1)
- R12 pad 1: +5V -> GND
- R12 pad 2: I2C1_SDA -> Net-(R12-Pad2)
- R13 pad 2: I2C1_SCL -> I2C1_SDA
- R2 pad 1: BOOT1 -> Net-(D1-Pad2)
- R2 pad 2: GND -> +3V3
- R3 pad 1: BOOT0 -> BOOT1
- R4 pad 1: Net-(D2-Pad2) -> BOOT0
- R4 pad 2: +3V3 -> GND
- R5 pad 1: +3V3 -> Net-(D2-Pad2)
- R5 pad 2: NRST -> +3V3
- R6 pad 1: +5V -> +3V3
- R6 pad 2: Net-(Q1-Pad1) -> NRST
- R7 pad 1: SIDE_SWITCH -> +5V
- R7 pad 2: GNDREF -> Net-(Q1-Pad1)
- R8 pad 1: GND -> SIDE_SWITCH
- R8 pad 2: Net-(R8-Pad2) -> GNDREF
- USB1 pad A4: Net-(FB2-Pad1) -> Net-(FB3-Pad1)
- USB1 pad A5: Net-(R8-Pad2) -> Net-(R9-Pad2)
- USB1 pad A9: Net-(FB2-Pad1) -> Net-(FB3-Pad1)
- USB1 pad B4: Net-(FB2-Pad1) -> Net-(FB3-Pad1)
- USB1 pad B5: Net-(R11-Pad2) -> Net-(R12-Pad2)
- USB1 pad B9: Net-(FB2-Pad1) -> Net-(FB3-Pad1)
- USB2 pad A5: Net-(R9-Pad2) -> Net-(R10-Pad2)
- USB2 pad B5: Net-(R9-Pad2) -> Net-(R10-Pad2)
- USB3 pad A5: Net-(R10-Pad2) -> Net-(R11-Pad2)
- USB3 pad B5: Net-(R10-Pad2) -> Net-(R11-Pad2)
- Y1 pad 2: HSE_IN -> (no net)
- Y1 pad 3: (no net) -> Net-(C8-Pad1)
Other:
- board text added: "See layout in AN2867"

Commit message: PAUSED: Use `git resume` to continue working.
Parts:
- removed the C10 at (-7.62, -0.51)
- removed the C12 at (25.4, 7.62)
- removed the C16 at (45.7, 29.2)
- removed the R1 at (-5.59, 1.27)
- removed R14: 2.7K, Resistor_SMD:R_0603_1608Metric
- removed the R8 at (-17.8, 53.3)
- added C11: 100n, Capacitor_SMD:C_0402_1005Metric, F.Cu at (4.45, -5.33)
- added C13: 100p, Capacitor_SMD:C_0402_1005Metric, F.Cu at (-1.91, 10.2)
- added C18: 10n, Capacitor_SMD:C_0402_1005Metric, F.Cu at (-17.4, -2.54)
- added R6: 10k, Resistor_SMD:R_0402_1005Metric, F.Cu at (-8.38, 3.43)
- added R9: 200k, Resistor_SMD:R_0402_1005Metric, F.Cu at (-21.6, 6.35)
- C14: value 100p -> 1u
- C15: value 4u7 -> 1u; footprint Capacitor_SMD:C_0603_1608Metric -> Capacitor_SMD:C_0402_1005Metric
- C17: value 10n -> 4u7; footprint Capacitor_SMD:C_0402_1005Metric -> Capacitor_SMD:C_0603_1608Metric
- C2: value 4u7 -> 10u
- C6: value 100n -> 6.8p
- C7: value 15p -> 6.8p
- C8, C9: value 15p -> 2.7p
- R11: value 200k -> 5.1K
- R12: value 5.1K -> 2.7K; footprint Resistor_SMD:R_0402_1005Metric -> Resistor_SMD:R_0603_1608Metric
- U2: value AMS1117-3.3 -> SOT-23-3 LDO; footprint Package_TO_SOT_SMD:SOT-223-3_TabPin2 -> Package_TO_SOT_SMD:SOT-23
- Y1: value 25MHz 12pF -> 25MHz 9pF; footprint Crystal:Crystal_SMD_3225-4Pin_3.2x2.5mm -> Crystal:Crystal_SMD_2520-4Pin_2.5x2.0mm
- Y2: value 32.768K 12.5p -> 32.768K 7p; footprint Crystal:Crystal_SMD_3215-2Pin_3.2x1.5mm -> Crystal:Crystal_SMD_2012-2Pin_2.0x1.2mm
- moved R11 81.9 mm to (-6.00, -11.0), turned to 90 degrees
- moved R10 76.5 mm to (11.7, 4.19), turned to 270 degrees
- moved J1 71.7 mm to (-30.5, -7.37)
- moved C17 66.0 mm to (-17.0, -3.94)
- moved C14 60.5 mm to (-8.26, -6.99), turned to 180 degrees
- moved R7 51.5 mm to (4.37, 8.89), turned to 270 degrees
- moved FB2 51.3 mm to (-3.17, 10.7), turned to 90 degrees
- moved C3 50.9 mm to (-3.30, -4.83), turned to 180 degrees
- moved C4 50.1 mm to (-4.83, 4.72)
- moved USB3 50.0 mm to (12.0, 12.0), turned to 30 degrees
- moved USB2 49.3 mm to (-12.0, 12.0), turned to 330 degrees
- moved Q1 48.6 mm to (-9.02, 1.02), turned to 180 degrees
- moved U2 45.7 mm to (-7.46, -4.64), turned to 0 degrees
- moved C6 45.5 mm to (5.21, -0.89), turned to 90 degrees
- moved C2 45.3 mm to (-5.00, 2.62), turned to 90 degrees
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- renumbered C11 to C10, C13 to C12, C18 to C16, R2 to R1, R3 to R2, R4 to R3, R5 to R4, R6 to R5, R9 to R8
Connections:
- C14 pad 1: Net-(C14-Pad1) -> +5V
- C14 pad 2: GNDREF -> GND
- C15 pad 1: +5V -> +3V3
- C17 pad 1: +3V3 -> (no net)
- C17 pad 2: GND -> (no net)
- C6 pad 1: +3V3 -> HSE_OUT
- C7 pad 1: HSE_OUT -> HSE_IN
- C8 pad 1: Net-(C8-Pad1) -> LSE_IN
- C9 pad 1: LSE_IN -> LSE_OUT
- FB2 pad 2: Net-(C14-Pad1) -> Net-(C13-Pad1)
- Q1 pad 3: Net-(C14-Pad1) -> Net-(C13-Pad1)
- Q2 pad 2: GNDREF -> GND
- R12 pad 1: GND -> +5V
- R12 pad 2: Net-(R12-Pad2) -> I2C1_SDA
- R13 pad 2: I2C1_SDA -> I2C1_SCL
- R7 pad 1: +5V -> SIDE_SWITCH
- R7 pad 2: Net-(Q1-Pad1) -> GND
- USB1 pad B5: Net-(R12-Pad2) -> Net-(R11-Pad2)
- USB2 pad A5: Net-(R10-Pad2) -> Net-(R9-Pad2)
- USB2 pad B5: Net-(R10-Pad2) -> Net-(R9-Pad2)
- USB3 pad A5: Net-(R11-Pad2) -> Net-(R10-Pad2)
- USB3 pad B5: Net-(R11-Pad2) -> Net-(R10-Pad2)
- Y1 pad 2: (no net) -> GND
- Y1 pad 3: Net-(C8-Pad1) -> HSE_IN
- Y1 pad 4: (no net) -> GND
Routing:
- net GND: track 0.00 -> 46.6 mm, vias 0 -> 37
- net Net-(FB3-Pad1): track 0.00 -> 34.4 mm
- net DP: track 0.00 -> 17.3 mm
- net DN: track 0.00 -> 15.8 mm
- net +3V3: track 0.00 -> 15.4 mm, vias 0 -> 2
- net HSE_IN: track 0.00 -> 8.23 mm
- net +3.3VA: track 0.00 -> 6.88 mm
- net Net-(R8-Pad2): track 0.00 -> 6.27 mm
- net LSE_OUT: track 0.00 -> 5.96 mm
- net Net-(R11-Pad2): track 0.00 -> 5.93 mm
- net +5V: track 0.00 -> 3.51 mm
- net HSE_OUT: track 0.00 -> 3.44 mm
- net LSE_IN: track 0.00 -> 2.86 mm
- net BOOT1: track 0.00 -> 1.25 mm
- added copper zone on F.Cu, net +3V3
- added copper zone on B.Cu, net GND
Other:
- board outline added: 30 x 30 mm
- board text removed: "See layout in AN2867"

Commit message: PAUSED: Use `git resume` to continue working.
Parts:
- removed C1, C11, C12, C16, C19, C3, C4, C5: 100n, Capacitor_SMD:C_0402_1005Metric
- removed C10, C14, C15: 1u, Capacitor_SMD:C_0402_1005Metric
- removed C13: 100p, Capacitor_SMD:C_0402_1005Metric
- removed C17: 4u7, Capacitor_SMD:C_0603_1608Metric
- removed C18: 10n, Capacitor_SMD:C_0402_1005Metric
- removed C2: 10u, Capacitor_SMD:C_0603_1608Metric
- removed C6, C7: 6.8p, Capacitor_SMD:C_0402_1005Metric
- removed C8, C9: 2.7p, Capacitor_SMD:C_0402_1005Metric
- removed D1: Red LED, LED_SMD:LED_0603_1608Metric
- removed D2: Blue LED, LED_SMD:LED_0603_1608Metric
- removed FB1, FB2, FB3: 470 @ 100MHz, Inductor_SMD:L_0603_1608Metric
- removed J1: Conn_01x04_Female, Connector_PinHeader_2.54mm:PinHeader_1x04_P2.54mm_Vertical
- removed Q1: Q_PMOS_GSD, -3.6A 0.02R, Package_TO_SOT_SMD:SOT-23
- removed Q2: Q_NMOS_GSD 1Amp, Package_TO_SOT_SMD:SOT-23
- removed R1: 5.1K, Resistor_SMD:R_0603_1608Metric
- removed R10, R9: 200k, Resistor_SMD:R_0402_1005Metric
- removed R11, R8: 5.1K, Resistor_SMD:R_0402_1005Metric
- removed R12, R13: 2.7K, Resistor_SMD:R_0603_1608Metric
- removed R2, R3, R5, R6, R7: 10k, Resistor_SMD:R_0402_1005Metric
- removed R4: 1.5K, Resistor_SMD:R_0603_1608Metric
- removed SW1, SW2: SW_SPST, Common:K2-1102SP-C4SC-04
- removed U1: STM32F411CEUx, Package_DFN_QFN:QFN-48-1EP_7x7mm_P0.5mm_EP5.6x5.6mm
- removed U2: SOT-23-3 LDO, Package_TO_SOT_SMD:SOT-23
- removed U3: 24LC256, Package_SO:SOIC-8_3.9x4.9mm_P1.27mm
- removed USB1, USB2, USB3: USB_C_Receptacle_USB2.0, Connector_USB:USB_C_Receptacle_HRO_TYPE-C-31-M-12
- removed Y1: 25MHz 9pF, Crystal:Crystal_SMD_2520-4Pin_2.5x2.0mm
- removed Y2: 32.768K 7p, Crystal:Crystal_SMD_2012-2Pin_2.0x1.2mm
Routing:
- net GND: track 46.6 -> 0.00 mm, vias 37 -> 0
- net Net-(FB3-Pad1): track 34.4 -> 0.00 mm
- net DP: track 17.3 -> 0.00 mm
- net DN: track 15.8 -> 0.00 mm
- net +3V3: track 15.4 -> 0.00 mm, vias 2 -> 0
- net HSE_IN: track 8.23 -> 0.00 mm
- net +3.3VA: track 6.88 -> 0.00 mm
- net Net-(R8-Pad2): track 6.27 -> 0.00 mm
- net LSE_OUT: track 5.96 -> 0.00 mm
- net Net-(R11-Pad2): track 5.93 -> 0.00 mm
- net +5V: track 3.51 -> 0.00 mm
- net HSE_OUT: track 3.44 -> 0.00 mm
- net LSE_IN: track 2.86 -> 0.00 mm
- net BOOT1: track 1.25 -> 0.00 mm
- removed copper zone on F.Cu, net +3V3
- removed copper zone on B.Cu, net GND
Other:
- board outline removed

Commit message: PAUSED: Use `git resume` to continue working.
Parts:
- added C1: 100n, Capacitor_SMD:C_0402_1005Metric, F.Cu at (-3.23, 4.67)
- added C10: 1u, Capacitor_SMD:C_0402_1005Metric, F.Cu at (1.93, 5.13)
- added C11: 100n, Capacitor_SMD:C_0402_1005Metric, F.Cu at (2.95, 5.13)
- added C12: 100n, Capacitor_SMD:C_0402_1005Metric, F.Cu at (-15.3, -10.6)
- added C13: 100p, Capacitor_SMD:C_0402_1005Metric, F.Cu at (11.7, 3.89)
- added C14: 1u, Capacitor_SMD:C_0402_1005Metric, F.Cu at (8.31, -5.59)
- added C15: 1u, Capacitor_SMD:C_0402_1005Metric, F.Cu at (3.71, -5.16)
- added C16: 100n, Capacitor_SMD:C_0402_1005Metric, F.Cu at (-13.0, -14.9)
- added C19: 100n, Capacitor_SMD:C_0402_1005Metric, F.Cu at (3.35, 15.2)
- added C2: 10u, Capacitor_SMD:C_0603_1608Metric, F.Cu at (-3.99, -4.93)
- added C3: 100n, Capacitor_SMD:C_0402_1005Metric, F.Cu at (-3.43, -6.20)
- added C4: 100n, Capacitor_SMD:C_0402_1005Metric, F.Cu at (-4.67, 3.23)
- added C5: 100n, Capacitor_SMD:C_0402_1005Metric, F.Cu at (4.67, -2.29)
- added C6: 6.8p, Capacitor_SMD:C_0402_1005Metric, F.Cu at (1.62, 8.92)
- added C7: 6.8p, Capacitor_SMD:C_0402_1005Metric, F.Cu at (1.62, 13.4)
- added C8: 2.7p, Capacitor_SMD:C_0402_1005Metric, F.Cu at (-3.30, 9.32)
- added C9: 2.7p, Capacitor_SMD:C_0402_1005Metric, F.Cu at (-3.30, 13.0)
- added D1: Red LED, LED_SMD:LED_0603_1608Metric, F.Cu at (-10.6, -17.3)
- added D2: Blue LED, LED_SMD:LED_0603_1608Metric, F.Cu at (-9.98, -8.66)
- added FB1: 470 @ 100MHz, Inductor_SMD:L_0603_1608Metric, F.Cu at (4.24, 5.69)
- added FB2: 470 @ 100MHz, Inductor_SMD:L_0603_1608Metric, F.Cu at (9.14, 4.06)
- added FB3: 470 @ 100MHz, Inductor_SMD:L_0603_1608Metric, F.Cu at (6.25, -8.75)
- added J1: Conn_01x04_Female, Connector_PinHeader_2.54mm:PinHeader_1x04_P2.54mm_Vertical, F.Cu at (22.9, -20.5)
- added Q1: Q_PMOS_GSD, -3.6A 0.02R, Package_TO_SOT_SMD:SOT-23, F.Cu at (10.0, 1.43)
- added Q2: Q_NMOS_GSD 1Amp, Package_TO_SOT_SMD:SOT-23, F.Cu at (10.0, -2.32)
- added R1: 5.1K, Resistor_SMD:R_0603_1608Metric, F.Cu at (-10.5, -19.1)
- added R10: 200k, Resistor_SMD:R_0402_1005Metric, F.Cu at (21.2, 14.9)
- added R11: 5.1K, Resistor_SMD:R_0402_1005Metric, F.Cu at (7.47, -19.4)
- added R12: 2.7K, Resistor_SMD:R_0603_1608Metric, F.Cu at (12.4, 8.89)
- added R13: 2.7K, Resistor_SMD:R_0603_1608Metric, F.Cu at (14.2, 8.89)
- added R2: 10k, Resistor_SMD:R_0402_1005Metric, F.Cu at (4.67, 0.00)
- added R3: 10k, Resistor_SMD:R_0402_1005Metric, F.Cu at (-14.6, -8.69)
- added R4: 1.5K, Resistor_SMD:R_0603_1608Metric, F.Cu at (-10.1, -10.6)
- added R5: 10k, Resistor_SMD:R_0402_1005Metric, F.Cu at (-13.4, -17.4)
- added R6: 10k, Resistor_SMD:R_0402_1005Metric, F.Cu at (12.5, 1.14)
- added R7: 10k, Resistor_SMD:R_0402_1005Metric, F.Cu at (12.3, -1.50)
- added R8: 5.1K, Resistor_SMD:R_0402_1005Metric, F.Cu at (8.26, -21.3)
- added R9: 200k, Resistor_SMD:R_0402_1005Metric, F.Cu at (-21.1, 13.8)
- added SW1: SW_SPST, Button_Switch_SMD:SW_SPST_B3U-1000P, F.Cu at (-18.0, -9.47)
- added SW2: SW_SPST, Button_Switch_SMD:SW_SPST_B3U-1000P, F.Cu at (-16.7, -15.1)
- added U1: STM32F411CEUx, Package_DFN_QFN:QFN-48-1EP_7x7mm_P0.5mm_EP5.6x5.6mm, F.Cu at (0.00, 0.00)
- added U2: SOT-23-3 LDO, Package_TO_SOT_SMD:SOT-23, F.Cu at (6.00, -6.00)
- added U3: 24LC256, Package_SO:SOIC-8_3.9x4.9mm_P1.27mm, F.Cu at (-1.00, 17.3)
- added USB1: USB_C_Receptacle_USB2.0, Connector_USB:USB_C_Receptacle_HRO_TYPE-C-31-M-12, F.Cu at (0.00, -21.0)
- added USB2: USB_C_Receptacle_USB2.0, Connector_USB:USB_C_Receptacle_HRO_TYPE-C-31-M-12, F.Cu at (-19.5, 21.0)
- added USB3: USB_C_Receptacle_USB2.0, Connector_USB:USB_C_Receptacle_HRO_TYPE-C-31-M-12, F.Cu at (19.0, 21.0)
- added Y1: 25MHz 9pF, Crystal:Crystal_SMD_2520-4Pin_2.5x2.0mm, F.Cu at (1.62, 11.2)
- added Y2: 32.768K 7p, Crystal:Crystal_SMD_2012-2Pin_2.0x1.2mm, F.Cu at (-3.30, 11.2)
Routing:
- net +5V: track 0.00 -> 17.4 mm
- net +3V3: track 0.00 -> 13.2 mm
- net Net-(FB3-Pad1): track 0.00 -> 9.23 mm
- net HSE_IN: track 0.00 -> 8.74 mm
- net LSE_OUT: track 0.00 -> 5.87 mm
- net HSE_OUT: track 0.00 -> 5.41 mm
- net LSE_IN: track 0.00 -> 4.39 mm
- net I2C1_SDA: track 0.00 -> 2.80 mm
- net +3.3VA: track 0.00 -> 2.50 mm
- net GND: track 0.00 -> 2.16 mm, vias 0 -> 5
- net I2C1_SCL: track 0.00 -> 2.03 mm
- added copper zone on B.Cu, net GND
Other:
- board outline added: 50 x 50 mm
