File: Synapse.kicad_pcb (KiCad board)
At the start: 2 copper layers, 50 x 50 mm, 48 parts, among them J1 Conn_01x04_Female, Q1 Q_PMOS_GSD, -3.6A 0.02R, Q2 Q_NMOS_GSD 1Amp, SW1 SW_SPST, SW2 SW_SPST, U1 STM32F411CEUx, U2 SOT-23-3 LDO, U3 24LC256, Y1 25MHz 9pF, Y2 32.768K 7p

Commit message: PAUSED: Use `git resume` to continue working.
Parts:
- moved C19 20.6 mm to (-6.65, -2.79)
- moved U3 20.6 mm to (-11.0, -0.73)
Routing:
- net +5V: track 17.4 -> 0.00 mm
- net +3V3: track 13.2 -> 0.00 mm
- net Net-(FB3-Pad1): track 9.23 -> 0.24 mm
- net SWDIO: track 0.00 -> 3.72 mm, vias 0 -> 1
- net DN: track 0.00 -> 2.13 mm, vias 0 -> 1
- net DP: track 0.00 -> 1.19 mm, vias 0 -> 1
Changed lines of the file:
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@@
   (general
     (thickness 1.6002)
-    (drawings 4)
-    (tracks 50)
+    (drawings 6)
+    (tracks 52)
     (zones 0)
     (modules 48)
@@
     (solder_mask_min_width 0.12)
     (aux_axis_origin 0 0)
-    (grid_origin 8.382 -8.128)
     (visible_elements FEFFFFFF)
     (pcbplotparams
@@
   )
   (module Package_SO:SOIC-8_3.9x4.9mm_P1.27mm (layer Front)
-    (at -1 17.272)
+    (at -11 -0.728)
     (descr "SOIC, 8 Pin (JEDEC MS-012AA, https://www.analog.com/media/en/package-pcb-resources/package/pkg_pdf/soic_narrow-r/r_8.pdf), generated with kicad-footprint-generator ipc_gullwing_generator.py")
     (tags "SOIC SO")
@@
   )
   (module Capacitor_SMD:C_0402_1005Metric (layer Front)
-    (at 3.3528 15.212 90)
+    (at -6.6472 -2.788 90)
     (descr "Capacitor SMD 0402 (1005 Metric), square (rectangular) end terminal, IPC_7351 nominal, (Body size source: IPC-SM-782 page 76, https://www.pcb-3d.com/wordpress/wp-content/uploads/ipc-sm-782a_amendment_1_and_2.pdf), generated with kicad-footprint-generator")
     (tags capacitor)
@@
     )
   )
+  (gr_poly (pts (xy 63.382 7.872) (xy 33.382 7.872) (xy 33.382 -25.128) (xy 63.382 -25.128)) (layer Cmts.User) (width 0.1))
+  (gr_poly (pts (xy 64.382 7.872) (xy 34.382 -25.128) (xy 64.382 -25.128)) (layer Cmts.User) (width 0.1))
   (gr_line (start 25 -25) (end 25 25) (layer Edge.Cuts) (width 0.1))
   (gr_line (start -25 -25) (end 25 -25) (layer Edge.Cuts) (width 0.1))
@@
   (segment (start -2.822 9.258) (end -2.327 8.763) (width 0.6) (layer Front) (net 1))
   (segment (start -2.822 9.3218) (end -2.822 9.258) (width 0.6) (layer Front) (net 1))
-  (segment (start 5 -5.05) (end 5.364 -5.05) (width 0.6) (layer Front) (net 2))
-  (segment (start 5.364 -5.05) (end 5.842 -4.572) (width 0.6) (layer Front) (net 2))
-  (segment (start 5.842 -4.572) (end 5.842 7.62) (width 0.6) (layer Front) (net 2))
   (segment (start -0.25 3.4375) (end -0.25 5.719) (width 0.3) (layer Front) (net 3))
   (segment (start -0.25 9.148) (end 0.9144 10.3124) (width 0.3) (layer Front) (net 3))
@@
   (segment (start 1.25 3.9932) (end 1.905 4.6482) (width 0.3) (layer Front) (net 7))
   (segment (start 1.9304 4.6508) (end 2.9438 4.6508) (width 0.6) (layer Front) (net 7))
-  (segment (start 7 -6) (end 7 8.494) (width 0.6) (layer Front) (net 9))
-  (segment (start 7 -6) (end 7 -8.778) (width 0.6) (layer Front) (net 9))
-  (segment (start 7 -8.778) (end 7.112 -8.89) (width 0.6) (layer Front) (net 9))
+  (via (at -1.477003 -5.5) (size 0.6) (drill 0.3) (layers Front Back) (net 16))
+  (segment (start -1.827001 -5.150002) (end -1.477003 -5.5) (width 0.3) (layer Front) (net 16))
+  (segment (start -1.827001 -3.514501) (end -1.827001 -5.150002) (width 0.3) (layer Front) (net 16))
+  (segment (start -1.75 -3.4375) (end -1.827001 -3.514501) (width 0.3) (layer Front) (net 16))
+  (segment (start -1.477003 -5.5) (end -1.477003 -6.977003) (width 0.3) (layer Back) (net 16))
   (segment (start 19.121601 17.957001) (end 18.465001 17.957001) (width 0.3) (layer Front) (net 23))
   (segment (start 19.25 17.828602) (end 19.121601 17.957001) (width 0.3) (layer Front) (net 23))
@@
   (segment (start 19.621601 15.952999) (end 19.7866 16.117998) (width 0.3) (layer Front) (net 24))
   (segment (start 18.75 16.955) (end 18.75 16.081398) (width 0.3) (layer Front) (net 24))
-  (segment (start 5.025 -8.75) (end 2.5 -11.275) (width 0.6) (layer Front) (net 27))
-  (segment (start 5.4625 -8.75) (end 5.025 -8.75) (width 0.6) (layer Front) (net 27))
+  (via (at -1.25 -4.625) (size 0.6) (drill 0.3) (layers Front Back) (net 25))
+  (segment (start -1.25 -3.4375) (end -1.25 -4.625) (width 0.3) (layer Front) (net 25))
+  (segment (start -0.672999 -5.422999) (end -0.75 -5.5) (width 0.3) (layer Front) (net 26))
+  (segment (start -0.672999 -3.514501) (end -0.672999 -5.422999) (width 0.3) (layer Front) (net 26))
+  (via (at -0.75 -5.5) (size 0.6) (drill 0.3) (layers Front Back) (net 26))
+  (segment (start -0.75 -3.4375) (end -0.672999 -3.514501) (width 0.3) (layer Front) (net 26))
   (segment (start 2.5 -16.25) (end 2.327001 -16.422999) (width 0.6) (layer Front) (net 27))
-  (segment (start 2.5 -11.275) (end 2.5 -16.25) (width 0.6) (layer Front) (net 27))
   (zone (net 1) (net_name GND) (layer Back) (hatch edge 0.508)
     (connect_pads (clearance 0.508))

Commit message: PAUSED: Use `git resume` to continue working.
Parts:
- moved C13 28.8 mm to (-17.0, 6.48), turned to 270 degrees
- moved R13 27.9 mm to (-11.9, -0.76), turned to 0 degrees
- moved R7 27.4 mm to (-15.1, -2.29), turned to 180 degrees
- moved R6 25.8 mm to (-13.2, 3.17)
- moved Q2 25.7 mm to (-15.6, 0.00), turned to 270 degrees
- moved Q1 25.7 mm to (-15.6, 3.56)
- moved R12 25.6 mm to (-11.9, 1.02), turned to 0 degrees
- moved FB2 24.9 mm to (-15.6, 6.86), turned to 90 degrees
- moved D2 23.4 mm to (-30.8, -19.3)
- moved R4 23.4 mm to (-30.9, -21.3)
- moved SW2 22.3 mm to (-37.2, -23.7)
- moved C16 22.0 mm to (-33.9, -21.9)
- moved R5 22.0 mm to (-34.2, -24.4)
- moved D1 21.1 mm to (-30.9, -23.1)
- moved R1 21.1 mm to (-30.8, -24.9)
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Routing:
- net SWDIO: track 3.72 -> 0.00 mm, vias 1 -> 0
- net I2C1_SDA: track 2.80 -> 0.00 mm
- net GND: track 2.16 -> 0.00 mm, vias 5 -> 0
- net DN: track 2.13 -> 0.00 mm, vias 1 -> 0
- net I2C1_SCL: track 2.03 -> 0.00 mm
- net +3V3: track 0.00 -> 1.32 mm, vias 0 -> 1
- net DP: track 1.19 -> 0.00 mm, vias 1 -> 0
Other:
- copper layers 2 -> 4
- net class Default: trace_width 0.127 -> 0.254
- net class GND removed
- rule trace_min: 0.127 -> 0.09
- rule via_min_drill: 0.3 -> 0.2
- rule via_min_size: 0.6 -> 0.4
