File: Synapse.kicad_pcb (KiCad board)
At the start: 4 copper layers, 40.7 x 42.5 mm, 46 parts, among them J1 SWD, Q1 Q_PMOS_GSD, -3.6A 0.02R, Q2 Q_NMOS_GSD 1Amp, SW1 SW_SPST, SW2 SW_SPST, U1 STM32F411CEUx, U2 SOT-23-3 LDO, U3 24LC256, Y1 25MHz 9pF, Y2 32.768K 7p

Commit message: PAUSED: Use `git resume` to continue working.
Parts:
- removed the R10 at (5.50, 16.0)
- added R8: 200k, Resistor_SMD:R_0402_1005Metric, F.Cu at (-5.50, 16.0)
- moved R9 11.0 mm to (5.50, 16.0), turned to 315 degrees
- renumbered C10 to C1, C8 to C10, C9 to C11, C14 to C13, C15 to C14, C13 to C15, C19 to C17, C11 to C2, C2 to C3, C3 to C4, C4 to C5, C5 to C6, C1 to C7, C6 to C8, C7 to C9, R2 to R1, R11 to R10, R12 to R11, R13 to R12, R1 to R2, R6 to R4, R7 to R6, R8 to R7
Connections:
- USB2 pad A5: Net-(R9-Pad2) -> Net-(R8-Pad2)
- USB2 pad B5: Net-(R9-Pad2) -> Net-(R8-Pad2)
- USB3 pad A5: Net-(R10-Pad2) (its old number) -> Net-(R9-Pad2)
- USB3 pad B5: Net-(R10-Pad2) (its old number) -> Net-(R9-Pad2)
Routing:
- net Net-(R10-Pad2) (its old number): track 12.4 -> 0.00 mm
- net Net-(R8-Pad2): track 0.00 -> 11.9 mm
- net GND: track 101.3 -> 102.0 mm, vias 68 -> 70
- net Net-(R9-Pad2): track 11.9 -> 12.4 mm

Commit message: PAUSED: Use `git resume` to continue working.
Routing:
- net GND: vias 70 -> 86

Commit message: PAUSED: Use `git resume` to continue working.
Routing:
- net GND: vias 86 -> 75
Other:
- board text added: "3V3"
- board text added: "CLK"
- board text added: "DIO"
- board text added: "GND"

Commit message: PAUSED: Use `git resume` to continue working.
Other:
- board text added: "BOOT"
- board text added: "Dygma Raise Synapse V2.0"
- board text added: "RESET"
Changed lines of the file:
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@@
   (general
     (thickness 1.6002)
-    (drawings 12)
+    (drawings 15)
     (tracks 499)
     (zones 0)
@@
   (layers
     (0 Front signal)
-    (1 In1.Cu signal)
-    (2 In2.Cu signal)
+    (1 In1.Cu signal hide)
+    (2 In2.Cu signal hide)
     (31 Back signal)
-    (34 B.Paste user)
-    (35 F.Paste user)
+    (34 B.Paste user hide)
+    (35 F.Paste user hide)
     (36 B.SilkS user)
-    (37 F.SilkS user)
-    (38 B.Mask user)
-    (39 F.Mask user)
+    (37 F.SilkS user hide)
+    (38 B.Mask user hide)
+    (39 F.Mask user hide)
     (44 Edge.Cuts user)
-    (45 Margin user)
-    (46 B.CrtYd user)
-    (47 F.CrtYd user)
-    (49 F.Fab user)
+    (45 Margin user hide)
+    (46 B.CrtYd user hide)
+    (47 F.CrtYd user hide)
+    (49 F.Fab user hide)
   )
   (setup
@@
     (uvia_min_size 0.4)
     (uvia_min_drill 0.2)
-    (edge_width 0.038)
+    (edge_width 0.1)
     (segment_width 0.254)
-    (pcb_text_width 0.3048)
-    (pcb_text_size 1.524 1.524)
-    (mod_edge_width 0.1524)
-    (mod_text_size 0.8128 0.8128)
-    (mod_text_width 0.1524)
+    (pcb_text_width 0.153)
+    (pcb_text_size 0.8 0.8)
+    (mod_edge_width 0.153)
+    (mod_text_size 0.8 0.8)
+    (mod_text_width 0.153)
     (pad_size 0.25 0.875)
     (pad_drill 0)
@@
     )
   )
+  (gr_text "Dygma Raise\nSynapse V2.0" (at 0 -8) (layer B.SilkS)
+    (effects (font (size 0.8 0.8) (thickness 0.153)) (justify mirror))
+  )
+  (gr_text BOOT (at -7.125 3.75 90) (layer F.SilkS)
+    (effects (font (size 0.8 0.8) (thickness 0.153)))
+  )
+  (gr_text RESET (at -7.125 0.25 90) (layer F.SilkS)
+    (effects (font (size 0.8 0.8) (thickness 0.153)))
+  )
   (gr_text GND (at -3.875 20.125) (layer B.SilkS)
-    (effects (font (size 0.8128 0.8128) (thickness 0.1524)) (justify mirror))
+    (effects (font (size 0.8 0.8) (thickness 0.153)) (justify mirror))
   )
   (gr_text DIO (at -1.25 20.125) (layer B.SilkS)
-    (effects (font (size 0.8128 0.8128) (thickness 0.1524)) (justify mirror))
+    (effects (font (size 0.8 0.8) (thickness 0.153)) (justify mirror))
   )
   (gr_text CLK (at 1.25 20.125) (layer B.SilkS)
-    (effects (font (size 0.8128 0.8128) (thickness 0.1524)) (justify mirror))
+    (effects (font (size 0.8 0.8) (thickness 0.153)) (justify mirror))
   )
   (gr_text 3V3 (at 3.875 20.125) (layer B.SilkS)
-    (effects (font (size 0.8128 0.8128) (thickness 0.1524)) (justify mirror))
+    (effects (font (size 0.8 0.8) (thickness 0.153)) (justify mirror))
   )
   (gr_line (start -9.65 22.35) (end 9.65 22.35) (layer Edge.Cuts) (width 0.1))
