File: Synapse.kicad_pcb (KiCad board)
At the start: 4 copper layers, 40.7 x 42.5 mm, 41 parts, among them J1 SWD, J2 I2C, SW1 SW_SPST, SW2 SW_SPST, U1 STM32F411CEUx, U2 SOT-553 LDO, U3 24LC256, Y1 24MHz 8pF, Y2 32.768K 7p

Commit message: PAUSED: Use `git resume` to continue working.
Parts:
- added C17: 470p, Capacitor_SMD:C_0402_1005Metric, F.Cu at (13.7, -9.10)
- C1, C8: value 1u -> 10u
- FB1, FB2: footprint Inductor_SMD:L_0402_1005Metric -> Inductor_SMD:L_0603_1608Metric
- U2: value SOT-553 LDO -> SOT-23-5 LDO (LM8805); footprint Package_TO_SOT_SMD:SOT-553 -> Package_TO_SOT_SMD:SOT-23-5
- moved U2 10.5 mm to (12.0, -6.20)
- moved C1 7.65 mm to (11.4, -10.1)
- moved C8 7.65 mm to (11.4, -9.00)
- moved FB1 3.25 mm to (6.00, -10.8), turned to 90 degrees
- moved FB2 0.64 mm to (7.90, 0.55)
Connections:
- C1 pad 1: +5V -> GND
- C1 pad 2: GND -> +5V
- U2 pad 1: GND -> +5V
- U2 pad 2: +3V3 -> GND
- U2 pad 3: +5V -> (no net)
- U2 pad 4: (no net) -> Net-(C17-Pad1)
- U2 pad 5: (no net) -> +3V3
Routing:
- net +5V: track 75.2 -> 71.8 mm, vias 5 -> 4
- net GND: track 91.1 -> 88.7 mm, vias 28 -> 25
- net +3V3: track 29.7 -> 27.6 mm
- net Net-(FB1-Pad2): track 9.20 -> 8.35 mm
- net +3.3VA: track 7.53 -> 8.19 mm
Other:
- board text added: "Need more vias from 5v to the bus… .5A, so need like 3-4 vias"

Commit message: PAUSED: Use `git resume` to continue working.
Parts:
- moved J1 17.3 mm to (1.32, 27.9)
- moved J2 17.3 mm to (1.32, 30.5)
- moved R3 13.5 mm to (16.6, 4.23)
- moved R5 13.5 mm to (15.5, 4.23)
- moved U2 10.2 mm to (2.01, -8.25), turned to 270 degrees
- moved C17 8.85 mm to (4.89, -8.25)
- moved C10 7.61 mm to (4.32, 11.6)
- moved C1 6.96 mm to (4.45, -9.75), turned to 270 degrees
- moved C8 6.77 mm to (4.89, -7.14)
- moved C16 3.64 mm to (8.89, 4.86), turned to 90 degrees
- moved R9 2.99 mm to (-8.38, 0.00), turned to 270 degrees
- moved C15 2.72 mm to (-9.40, 0.00), turned to 90 degrees
- moved R1 1.78 mm to (6.00, -16.8)
- moved SW1 1.74 mm to (6.10, 5.87), turned to 270 degrees
- moved SW2 1.74 mm to (-6.10, 5.87), turned to 270 degrees
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Routing:
- net GND: track 88.7 -> 25.0 mm, vias 25 -> 17
- net +5V: track 71.8 -> 14.8 mm, vias 4 -> 6
- net I2C1_SDA: track 59.3 -> 10.9 mm, vias 8 -> 0
- net I2C1_SCL: track 57.8 -> 11.3 mm, vias 5 -> 0
- net SWDIO: track 27.7 -> 0.00 mm, vias 1 -> 0
- net SWCLK: track 21.1 -> 0.00 mm, vias 1 -> 0
- net BOOT0: track 15.8 -> 0.00 mm
- net +3V3: track 27.6 -> 12.4 mm, vias 8 -> 3
- net NRST: track 11.3 -> 0.00 mm
- net Net-(R4-Pad2): track 15.7 -> 4.41 mm
- net Net-(R7-Pad2): track 15.9 -> 6.09 mm
- net +3.3VA: track 8.19 -> 0.00 mm
- net HSE_IN: track 6.56 -> 0.00 mm
- net LSE_IN: track 5.44 -> 0.00 mm
- net HSE_OUT: track 5.04 -> 0.00 mm
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- added copper zone on In2.Cu, net +5V
- added copper zone on In2.Cu, net Net-(FB1-Pad2)

Commit message: PAUSED: Use `git resume` to continue working.
Parts:
- removed C8: 10u, Capacitor_SMD:C_0402_1005Metric
- removed J2: I2C, Common:TestPoint_Pads_4x2.54_D1.5mm
- removed R8: 10k, Resistor_SMD:R_0402_1005Metric
- removed SW1: SW_SPST, Button_Switch_SMD:SW_SPST_B3U-1000P
- C1: value 10u -> 1u
- C17: value 470p -> 1u
- J1: footprint Common:TestPoint_Pads_4x2.54_D1.5mm -> Common:TestPoint_Pads_5x2.54_D1.5mm
- U2: value SOT-23-5 LDO (LM8805) -> SOT-23-3L LDO 200mA; footprint Package_TO_SOT_SMD:SOT-23-5 -> Package_TO_SOT_SMD:SOT-23
- moved R2 16.7 mm to (10.6, -16.1)
- moved SW2 12.9 mm to (6.78, 5.18), turned to 90 degrees
- moved R9 12.2 mm to (-20.4, -2.25)
- moved C15 12.2 mm to (-21.4, -2.25)
- moved FB1 9.15 mm to (-2.50, -9.25), turned to 180 degrees
- moved R6 7.00 mm to (-10.0, -8.00)
- moved D1 7.00 mm to (-12.7, -7.60)
- moved C17 5.01 mm to (-0.12, -8.37), turned to 90 degrees
- moved C16 3.95 mm to (6.08, 2.08), turned to 180 degrees
- moved R1 3.44 mm to (9.38, -16.1)
- moved FB2 2.21 mm to (6.58, -1.22), turned to 0 degrees
- moved R10 2.01 mm to (6.12, -2.62), turned to 0 degrees
- moved C2 1.70 mm to (7.13, -5.12)
- moved C1 1.44 mm to (4.88, -8.37)
- moved U3 1.25 mm to (0.00, 11.8), turned to 0 degrees
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Connections:
- C1 pad 1: GND -> +5V
- C1 pad 2: +5V -> GND
- C17 pad 1: Net-(C17-Pad1) -> +3V3
- J1 pad 2: SWCLK -> NRST
- J1 pad 3: SWDIO -> SWCLK
- J1 pad 4: +3V3 -> SWDIO
- U2 pad 1: +5V -> GND
- U2 pad 2: GND -> +3V3
- U2 pad 3: (no net) -> +5V
Routing:
- net +5V: track 14.8 -> 0.00 mm, vias 6 -> 0
- net GND: track 25.0 -> 10.6 mm, vias 17 -> 2
- net +3V3: track 12.4 -> 0.00 mm, vias 3 -> 0
- net DP: track 13.5 -> 3.97 mm, vias 2 -> 0
- net DN: track 12.6 -> 4.19 mm, vias 2 -> 0
- net NRST: track 0.00 -> 6.87 mm
- net Net-(R7-Pad2): track 6.09 -> 0.00 mm
- net +3.3VA: track 0.00 -> 5.66 mm
- net Net-(R1-Pad2): track 7.05 -> 2.45 mm
- net Net-(R4-Pad2): track 4.41 -> 0.00 mm
- net Net-(C17-Pad1): track 3.82 -> 0.00 mm
- net Net-(R2-Pad2): track 6.00 -> 2.45 mm
- net Net-(D1-Pad1): track 2.36 -> 0.00 mm
- net BOOT1: track 1.96 -> 0.00 mm
- net I2C1_SCL: track 11.3 -> 12.0 mm
Other:
- board size 40.7 x 42.5 mm -> 180.2 x 46.9 mm

Commit message: Final form
Parts:
- removed the C10 at (4.32, 11.6)
- removed the C11 at (-0.87, 5.35)
- removed the C12 at (-3.57, 6.00)
- removed C17: 1u, Capacitor_SMD:C_0402_1005Metric
- removed the C7 at (-2.87, -7.62)
- removed the FB1 at (-2.50, -9.25)
- removed the R6 at (-10.0, -8.00)
- removed the R7 at (6.38, 17.5)
- removed the U2 at (2.38, -8.87)
- added C2: 1u, Capacitor_SMD:C_0402_1005Metric, F.Cu at (-5.50, 8.00)
- added C3: 100n, Capacitor_SMD:C_0402_1005Metric, F.Cu at (4.69, 10.9)
- added C6: 100n, Capacitor_SMD:C_0402_1005Metric, F.Cu at (-2.90, -7.62)
- added C8: 6p, Capacitor_SMD:C_0402_1005Metric, F.Cu at (-0.87, 5.65)
- added C9: 6p, Capacitor_SMD:C_0402_1005Metric, F.Cu at (3.73, 5.15)
- added FB2: 470 @ 100MHz, Inductor_SMD:L_0603_1608Metric, F.Cu at (2.45, -9.88)
- added FB3: 470 @ 100MHz, Inductor_SMD:L_0603_1608Metric, F.Cu at (-2.45, -9.88)
- added R3: 1K, Resistor_SMD:R_0402_1005Metric, F.Cu at (5.40, -10.4)
- added R8: 200k, Resistor_SMD:R_0402_1005Metric, F.Cu at (7.75, 18.0)
- added U1: SOT-23-3L LDO 200mA, Package_TO_SOT_SMD:SOT-23, F.Cu at (-7.00, 5.50)
- C13: value 6p -> 2.7p
- moved C10 32.6 mm to (10.00, 6.67), turned to 270 degrees
- moved R2 30.7 mm to (8.98, 6.65), turned to 90 degrees
- moved C1 20.5 mm to (-7.50, 8.00), turned to 0 degrees
- moved R9 16.6 mm to (-6.00, -15.5), turned to 90 degrees
- moved D1 15.9 mm to (3.20, -7.50), turned to 180 degrees
- moved C4 14.9 mm to (-7.00, -0.25), turned to 90 degrees
- moved J1 13.8 mm to (0.00, 14.2)
- moved R4 11.7 mm to (7.10, 11.0), turned to 180 degrees
- moved R5 7.85 mm to (8.90, 8.45), turned to 180 degrees
- moved C13 7.39 mm to (-3.57, 6.00)
- moved R6 3.44 mm to (6.00, -15.5), turned to 90 degrees
- moved USB2 1.36 mm to (-13.1, 14.7)
- moved USB3 1.36 mm to (13.1, 14.7)
- moved U2 1.00 mm to (0.00, 12.8)
- moved C5 0.64 mm to (5.50, -5.25)
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- renumbered C15 to C10, C5 to C11, C6 to C12, C3 to C15, C2 to C4, C4 to C5, C9 to C7, FB2 to FB1, R10 to R1, R9 to R2, R3 to R4, R1 to R6, R4 to R7, R2 to R9, SW2 to SW1, U3 to U2, U1 to U3
Connections:
- C13 pad 1: HSE_OUT -> LSE_IN
- J1 pad 2: NRST -> SWDIO
- J1 pad 4: SWDIO -> NRST
Routing:
- net GND: track 10.6 -> 79.7 mm, vias 2 -> 26
- net I2C1_SDA: track 11.0 -> 64.6 mm, vias 0 -> 8
- net I2C1_SCL: track 12.0 -> 62.0 mm, vias 0 -> 4
- net +3V3: track 0.00 -> 41.5 mm, vias 0 -> 8
- net SWDIO: track 0.00 -> 26.6 mm, vias 0 -> 1
- net SWCLK: track 0.00 -> 22.8 mm, vias 0 -> 1
- net BOOT0: track 0.00 -> 20.9 mm, vias 0 -> 2
- net +5V: track 0.00 -> 17.8 mm, vias 0 -> 7
- net Net-(R8-Pad2): track 0.00 -> 16.5 mm
- net Net-(R7-Pad2): track 0.00 -> 14.4 mm
- net NRST: track 6.87 -> 20.3 mm, vias 0 -> 1
- net HSE_IN: track 0.00 -> 7.57 mm
- net DP: track 3.97 -> 10.6 mm
- net Net-(FB2-Pad2): track 3.37 -> 9.23 mm
- net HSE_OUT: track 0.00 -> 5.60 mm
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- removed copper zone on In2.Cu, net Net-(FB2-Pad2)
Other:
- board size 180.2 x 46.9 mm -> 42 x 43.7 mm
- board text added: "RST"
- board text removed: "5V"
- board text removed: "Need more vias from 5v to the bus… .5A, so need like 3-4 vias"
- board text removed: "RESET"
- board text removed: "SCL"
- board text removed: "SDA"

Commit message: vegeta
Parts:
- moved C15 1.02 mm to (-6.05, 1.45), turned to 180 degrees
- moved C4 0.50 mm to (-7.00, -0.75)
- moved C7 0.50 mm to (-5.62, -0.12)
- moved C1 0.45 mm to (-7.50, 7.55)
- moved C2 0.45 mm to (-5.50, 7.55)
- moved U1 0.45 mm to (-7.00, 5.04)
Routing:
- net +3V3: track 41.5 -> 43.8 mm, vias 8 -> 9
- net GND: track 79.7 -> 77.5 mm
- net I2C1_SDA: track 64.6 -> 62.5 mm, vias 8 -> 9
- net +5V: track 17.8 -> 18.5 mm
- net I2C1_SCL: track 62.0 -> 62.3 mm, vias 4 -> 6

Commit message: New edge cuts
Other:
- board size 42 x 43.7 mm -> 41.3 x 42.8 mm
